File: kicad/esp32/IR_RCV.sch (KiCad schematic (older format))
At the start: 15 parts, among them P5 PR_Host, P6 PR_Slave, Q1 IRFML8244, U6 AD8601

Commit message: 自動配線成功
Parts:
- renumbered C19 to C14, C20 to C15, C21 to C16, P5 to P4, P6 to P5
Changed lines of the file:
@@
 $Descr A4 11693 8268
 encoding utf-8
-Sheet 4 13
+Sheet 4 14
 Title ""
 Date ""
@@
 $EndDescr
 $Comp
-L C C20
+L C C15
 U 1 1 57CF0F45
 P 5950 4200
-AR Path="/57CF0B09/57CF0F45" Ref="C20"  Part="1"
-AR Path="/57CF289D/57CF0F45" Ref="C23"  Part="1"
-AR Path="/57CF292E/57CF0F45" Ref="C26"  Part="1"
-AR Path="/57CF2A30/57CF0F45" Ref="C29"  Part="1"
-F 0 "C26" H 5975 4300 50  0000 L CNN
+AR Path="/57CF0B09/57CF0F45" Ref="C15"  Part="1"
+AR Path="/57CF289D/57CF0F45" Ref="C18"  Part="1"
+AR Path="/57CF292E/57CF0F45" Ref="C21"  Part="1"
+AR Path="/57CF2A30/57CF0F45" Ref="C24"  Part="1"
+F 0 "C15" H 5975 4300 50  0000 L CNN
 F 1 "0.01u" H 5975 4100 50  0000 L CNN
 F 2 "Capacitors_SMD:C_0201" H 5988 4050 50  0001 C CNN
@@
 AR Path="/57CF292E/57CF0F57" Ref="R19"  Part="1"
 AR Path="/57CF2A30/57CF0F57" Ref="R25"  Part="1"
-F 0 "R19" V 7030 3700 50  0000 C CNN
+F 0 "R7" V 7030 3700 50  0000 C CNN
 F 1 "220k" V 6950 3700 50  0000 C CNN
 F 2 "Resistors_SMD:R_0201" V 6880 3700 50  0001 C CNN
@@
 $EndComp
 $Comp
-L C C19
+L C C14
 U 1 1 57CF0F5E
 P 6950 3500
-AR Path="/57CF0B09/57CF0F5E" Ref="C19"  Part="1"
-AR Path="/57CF289D/57CF0F5E" Ref="C22"  Part="1"
-AR Path="/57CF292E/57CF0F5E" Ref="C25"  Part="1"
-AR Path="/57CF2A30/57CF0F5E" Ref="C28"  Part="1"
-F 0 "C25" H 6850 3600 50  0000 L CNN
+AR Path="/57CF0B09/57CF0F5E" Ref="C14"  Part="1"
+AR Path="/57CF289D/57CF0F5E" Ref="C17"  Part="1"
+AR Path="/57CF292E/57CF0F5E" Ref="C20"  Part="1"
+AR Path="/57CF2A30/57CF0F5E" Ref="C23"  Part="1"
+F 0 "C14" H 6850 3600 50  0000 L CNN
 F 1 "22p" H 6800 3400 50  0000 L CNN
 F 2 "Capacitors_SMD:C_0201" H 6988 3350 50  0001 C CNN
@@
 Connection ~ 7200 4100
 $Comp
-L CONN_01X04 P6
+L CONN_01X04 P5
 U 1 1 589BE652
 P 5400 2550
-AR Path="/57CF0B09/589BE652" Ref="P6"  Part="1"
-AR Path="/57CF289D/589BE652" Ref="P8"  Part="1"
-AR Path="/57CF292E/589BE652" Ref="P10"  Part="1"
-AR Path="/57CF2A30/589BE652" Ref="P12"  Part="1"
-F 0 "P10" H 5400 2800 50  0000 C CNN
+AR Path="/57CF0B09/589BE652" Ref="P5"  Part="1"
+AR Path="/57CF289D/589BE652" Ref="P7"  Part="1"
+AR Path="/57CF292E/589BE652" Ref="P9"  Part="1"
+AR Path="/57CF2A30/589BE652" Ref="P11"  Part="1"
+F 0 "P5" H 5400 2800 50  0000 C CNN
 F 1 "PR_Slave" V 5500 2550 50  0000 C CNN
 F 2 "mouse:STAND_PR_SLAVE" H 5400 2550 50  0001 C CNN
@@
 AR Path="/57CF292E/589BE75A" Ref="Q3"  Part="1"
 AR Path="/57CF2A30/589BE75A" Ref="Q4"  Part="1"
-F 0 "Q3" H 4600 4750 50  0000 R CNN
+F 0 "Q1" H 4600 4750 50  0000 R CNN
 F 1 "IRFML8244" H 4350 4900 50  0000 R CNN
 F 2 "TO_SOT_Packages_SMD:SOT-23" H 4500 4800 50  0001 C CNN
@@
 AR Path="/57CF292E/589BE766" Ref="D7"  Part="1"
 AR Path="/57CF2A30/589BE766" Ref="D9"  Part="1"
-F 0 "D7" H 4400 4200 50  0000 C CNN
+F 0 "D3" H 4400 4200 50  0000 C CNN
 F 1 "VSMB294008G" H 4400 3950 50  0000 C CNN
 F 2 "mouse:VISHAY_DIODE" H 4400 4100 50  0001 C CNN
@@
 AR Path="/57CF292E/589BE76D" Ref="R18"  Part="1"
 AR Path="/57CF2A30/589BE76D" Ref="R24"  Part="1"
-F 0 "R18" V 4480 3550 50  0000 C CNN
+F 0 "R6" V 4480 3550 50  0000 C CNN
 F 1 "100" V 4400 3550 50  0000 C CNN
 F 2 "Resistors_SMD:R_0402" V 4330 3550 50  0001 C CNN
@@
 AR Path="/57CF292E/589BE778" Ref="R23"  Part="1"
 AR Path="/57CF2A30/589BE778" Ref="R29"  Part="1"
-F 0 "R23" V 4080 4950 50  0000 C CNN
+F 0 "R11" V 4080 4950 50  0000 C CNN
 F 1 "10k" V 4000 4950 50  0000 C CNN
 F 2 "Resistors_SMD:R_0201" V 3930 4950 50  0001 C CNN
@@
 s_IR_LED
 $Comp
-L CONN_01X04 P5
+L CONN_01X04 P4
 U 1 1 589BE88F
 P 5000 2550
-AR Path="/57CF0B09/589BE88F" Ref="P5"  Part="1"
-AR Path="/57CF289D/589BE88F" Ref="P7"  Part="1"
-AR Path="/57CF292E/589BE88F" Ref="P9"  Part="1"
-AR Path="/57CF2A30/589BE88F" Ref="P11"  Part="1"
-F 0 "P9" H 5000 2800 50  0000 C CNN
+AR Path="/57CF0B09/589BE88F" Ref="P4"  Part="1"
+AR Path="/57CF289D/589BE88F" Ref="P6"  Part="1"
+AR Path="/57CF292E/589BE88F" Ref="P8"  Part="1"
+AR Path="/57CF2A30/589BE88F" Ref="P10"  Part="1"
+F 0 "P4" H 5000 2800 50  0000 C CNN
 F 1 "PR_Host" V 5100 2550 50  0000 C CNN
 F 2 "mouse:STAND_PR_HOST" H 5000 2550 50  0001 C CNN
@@
 AR Path="/57CF292E/589BEE35" Ref="D6"  Part="1"
 AR Path="/57CF2A30/589BEE35" Ref="D8"  Part="1"
-F 0 "D6" H 5600 4050 50  0000 C CNN
+F 0 "D2" H 5600 4050 50  0000 C CNN
 F 1 "VEMD2020X01" H 5600 3850 50  0000 C CNN
 F 2 "mouse:VISHAY_DIODE" H 5600 3950 50  0001 C CNN
@@
 AR Path="/57CF292E/589BEE3B" Ref="R22"  Part="1"
 AR Path="/57CF2A30/589BEE3B" Ref="R28"  Part="1"
-F 0 "R22" V 5680 4750 50  0000 C CNN
+F 0 "R10" V 5680 4750 50  0000 C CNN
 F 1 "100k" V 5600 4750 50  0000 C CNN
 F 2 "Resistors_SMD:R_0201" V 5530 4750 50  0001 C CNN
@@
 IR_LED
 $Comp
-L GND #PWR039
+L GND #PWR036
 U 1 1 589BF265
 P 4700 2800
-AR Path="/57CF0B09/589BF265" Ref="#PWR039"  Part="1"
-AR Path="/57CF289D/589BF265" Ref="#PWR041"  Part="1"
-AR Path="/57CF292E/589BF265" Ref="#PWR043"  Part="1"
-AR Path="/57CF2A30/589BF265" Ref="#PWR045"  Part="1"
-F 0 "#PWR045" H 4700 2550 50  0001 C CNN
+AR Path="/57CF0B09/589BF265" Ref="#PWR036"  Part="1"
+AR Path="/57CF289D/589BF265" Ref="#PWR038"  Part="1"
+AR Path="/57CF292E/589BF265" Ref="#PWR040"  Part="1"
+AR Path="/57CF2A30/589BF265" Ref="#PWR042"  Part="1"
+F 0 "#PWR042" H 4700 2550 50  0001 C CNN
 F 1 "GND" H 4700 2650 50  0000 C CNN
 F 2 "" H 4700 2800 50  0000 C CNN
@@
 	4700 2300 4700 2400
 $Comp
-L C C21
+L C C16
 U 1 1 589EE263
 P 4900 4750
-AR Path="/57CF0B09/589EE263" Ref="C21"  Part="1"
-AR Path="/57CF289D/589EE263" Ref="C24"  Part="1"
-AR Path="/57CF292E/589EE263" Ref="C27"  Part="1"
-AR Path="/57CF2A30/589EE263" Ref="C30"  Part="1"
-F 0 "C27" H 4925 4850 50  0000 L CNN
+AR Path="/57CF0B09/589EE263" Ref="C16"  Part="1"
+AR Path="/57CF289D/589EE263" Ref="C19"  Part="1"
+AR Path="/57CF292E/589EE263" Ref="C22"  Part="1"
+AR Path="/57CF2A30/589EE263" Ref="C25"  Part="1"
+F 0 "C16" H 4925 4850 50  0000 L CNN
 F 1 "47u" H 4925 4650 50  0000 L CNN
 F 2 "Capacitors_SMD:C_0805" H 4938 4600 50  0001 C CNN
@@
 	4700 2700 4700 2800
 $Comp
-L +3.3V #PWR040
+L +3.3V #PWR037
 U 1 1 589CC209
 P 4700 2300
-AR Path="/57CF0B09/589CC209" Ref="#PWR040"  Part="1"
-AR Path="/57CF289D/589CC209" Ref="#PWR042"  Part="1"
-AR Path="/57CF292E/589CC209" Ref="#PWR044"  Part="1"
-AR Path="/57CF2A30/589CC209" Ref="#PWR046"  Part="1"
-F 0 "#PWR046" H 4700 2150 50  0001 C CNN
+AR Path="/57CF0B09/589CC209" Ref="#PWR037"  Part="1"
+AR Path="/57CF289D/589CC209" Ref="#PWR039"  Part="1"
+AR Path="/57CF292E/589CC209" Ref="#PWR041"  Part="1"
+AR Path="/57CF2A30/589CC209" Ref="#PWR043"  Part="1"
+F 0 "#PWR043" H 4700 2150 50  0001 C CNN
 F 1 "+3.3V" H 4700 2440 50  0000 C CNN
 F 2 "" H 4700 2300 50  0000 C CNN
@@
 AR Path="/57CF292E/58A0483E" Ref="R20"  Part="1"
 AR Path="/57CF2A30/58A0483E" Ref="R26"  Part="1"
-F 0 "R20" V 6280 3750 50  0000 C CNN
+F 0 "R8" V 6280 3750 50  0000 C CNN
 F 1 "1k" V 6200 3750 50  0000 C CNN
 F 2 "Resistors_SMD:R_0201" V 6130 3750 50  0001 C CNN
@@
 AR Path="/57CF292E/58A04889" Ref="R21"  Part="1"
 AR Path="/57CF2A30/58A04889" Ref="R27"  Part="1"
-F 0 "R21" V 6280 4450 50  0000 C CNN
+F 0 "R9" V 6280 4450 50  0000 C CNN
 F 1 "1k" V 6200 4450 50  0000 C CNN
 F 2 "Resistors_SMD:R_0201" V 6130 4450 50  0001 C CNN
@@
 AR Path="/57CF292E/58A04D19" Ref="U8"  Part="1"
 AR Path="/57CF2A30/58A04D19" Ref="U9"  Part="1"
-F 0 "U8" H 6850 4300 50  0000 C CNN
+F 0 "U6" H 6850 4300 50  0000 C CNN
 F 1 "AD8601" H 7000 3900 50  0000 C CNN
 F 2 "TO_SOT_Packages_SMD:SOT-23-5" H 6750 4200 50  0001 C CNN

Commit message: 更新
Changed lines of the file:
@@
 AR Path="/57CF292E/57CF0F45" Ref="C21"  Part="1"
 AR Path="/57CF2A30/57CF0F45" Ref="C24"  Part="1"
-F 0 "C15" H 5975 4300 50  0000 L CNN
+F 0 "C24" H 5975 4300 50  0000 L CNN
 F 1 "0.01u" H 5975 4100 50  0000 L CNN
 F 2 "Capacitors_SMD:C_0201" H 5988 4050 50  0001 C CNN
@@
 AR Path="/57CF292E/57CF0F57" Ref="R19"  Part="1"
 AR Path="/57CF2A30/57CF0F57" Ref="R25"  Part="1"
-F 0 "R7" V 7030 3700 50  0000 C CNN
+F 0 "R25" V 7030 3700 50  0000 C CNN
 F 1 "220k" V 6950 3700 50  0000 C CNN
 F 2 "Resistors_SMD:R_0201" V 6880 3700 50  0001 C CNN
@@
 AR Path="/57CF292E/57CF0F5E" Ref="C20"  Part="1"
 AR Path="/57CF2A30/57CF0F5E" Ref="C23"  Part="1"
-F 0 "C14" H 6850 3600 50  0000 L CNN
+F 0 "C23" H 6850 3600 50  0000 L CNN
 F 1 "22p" H 6800 3400 50  0000 L CNN
 F 2 "Capacitors_SMD:C_0201" H 6988 3350 50  0001 C CNN
@@
 AR Path="/57CF292E/589BE652" Ref="P9"  Part="1"
 AR Path="/57CF2A30/589BE652" Ref="P11"  Part="1"
-F 0 "P5" H 5400 2800 50  0000 C CNN
+F 0 "P11" H 5400 2800 50  0000 C CNN
 F 1 "PR_Slave" V 5500 2550 50  0000 C CNN
 F 2 "mouse:STAND_PR_SLAVE" H 5400 2550 50  0001 C CNN
@@
 AR Path="/57CF292E/589BE75A" Ref="Q3"  Part="1"
 AR Path="/57CF2A30/589BE75A" Ref="Q4"  Part="1"
-F 0 "Q1" H 4600 4750 50  0000 R CNN
+F 0 "Q4" H 4600 4750 50  0000 R CNN
 F 1 "IRFML8244" H 4350 4900 50  0000 R CNN
 F 2 "TO_SOT_Packages_SMD:SOT-23" H 4500 4800 50  0001 C CNN
@@
 AR Path="/57CF292E/589BE766" Ref="D7"  Part="1"
 AR Path="/57CF2A30/589BE766" Ref="D9"  Part="1"
-F 0 "D3" H 4400 4200 50  0000 C CNN
+F 0 "D9" H 4400 4200 50  0000 C CNN
 F 1 "VSMB294008G" H 4400 3950 50  0000 C CNN
 F 2 "mouse:VISHAY_DIODE" H 4400 4100 50  0001 C CNN
@@
 AR Path="/57CF292E/589BE76D" Ref="R18"  Part="1"
 AR Path="/57CF2A30/589BE76D" Ref="R24"  Part="1"
-F 0 "R6" V 4480 3550 50  0000 C CNN
+F 0 "R24" V 4480 3550 50  0000 C CNN
 F 1 "100" V 4400 3550 50  0000 C CNN
 F 2 "Resistors_SMD:R_0402" V 4330 3550 50  0001 C CNN
@@
 AR Path="/57CF292E/589BE778" Ref="R23"  Part="1"
 AR Path="/57CF2A30/589BE778" Ref="R29"  Part="1"
-F 0 "R11" V 4080 4950 50  0000 C CNN
+F 0 "R29" V 4080 4950 50  0000 C CNN
 F 1 "10k" V 4000 4950 50  0000 C CNN
 F 2 "Resistors_SMD:R_0201" V 3930 4950 50  0001 C CNN
@@
 AR Path="/57CF292E/589BE88F" Ref="P8"  Part="1"
 AR Path="/57CF2A30/589BE88F" Ref="P10"  Part="1"
-F 0 "P4" H 5000 2800 50  0000 C CNN
+F 0 "P10" H 5000 2800 50  0000 C CNN
 F 1 "PR_Host" V 5100 2550 50  0000 C CNN
 F 2 "mouse:STAND_PR_HOST" H 5000 2550 50  0001 C CNN
@@
 AR Path="/57CF292E/589BEE35" Ref="D6"  Part="1"
 AR Path="/57CF2A30/589BEE35" Ref="D8"  Part="1"
-F 0 "D2" H 5600 4050 50  0000 C CNN
+F 0 "D8" H 5600 4050 50  0000 C CNN
 F 1 "VEMD2020X01" H 5600 3850 50  0000 C CNN
 F 2 "mouse:VISHAY_DIODE" H 5600 3950 50  0001 C CNN
@@
 AR Path="/57CF292E/589BEE3B" Ref="R22"  Part="1"
 AR Path="/57CF2A30/589BEE3B" Ref="R28"  Part="1"
-F 0 "R10" V 5680 4750 50  0000 C CNN
+F 0 "R28" V 5680 4750 50  0000 C CNN
 F 1 "100k" V 5600 4750 50  0000 C CNN
 F 2 "Resistors_SMD:R_0201" V 5530 4750 50  0001 C CNN
@@
 AR Path="/57CF292E/589EE263" Ref="C22"  Part="1"
 AR Path="/57CF2A30/589EE263" Ref="C25"  Part="1"
-F 0 "C16" H 4925 4850 50  0000 L CNN
+F 0 "C25" H 4925 4850 50  0000 L CNN
 F 1 "47u" H 4925 4650 50  0000 L CNN
 F 2 "Capacitors_SMD:C_0805" H 4938 4600 50  0001 C CNN
@@
 AR Path="/57CF292E/58A0483E" Ref="R20"  Part="1"
 AR Path="/57CF2A30/58A0483E" Ref="R26"  Part="1"
-F 0 "R8" V 6280 3750 50  0000 C CNN
+F 0 "R26" V 6280 3750 50  0000 C CNN
 F 1 "1k" V 6200 3750 50  0000 C CNN
 F 2 "Resistors_SMD:R_0201" V 6130 3750 50  0001 C CNN
@@
 AR Path="/57CF292E/58A04889" Ref="R21"  Part="1"
 AR Path="/57CF2A30/58A04889" Ref="R27"  Part="1"
-F 0 "R9" V 6280 4450 50  0000 C CNN
+F 0 "R27" V 6280 4450 50  0000 C CNN
 F 1 "1k" V 6200 4450 50  0000 C CNN
 F 2 "Resistors_SMD:R_0201" V 6130 4450 50  0001 C CNN
@@
 AR Path="/57CF292E/58A04D19" Ref="U8"  Part="1"
 AR Path="/57CF2A30/58A04D19" Ref="U9"  Part="1"
-F 0 "U6" H 6850 4300 50  0000 C CNN
+F 0 "U9" H 6850 4300 50  0000 C CNN
 F 1 "AD8601" H 7000 3900 50  0000 C CNN
 F 2 "TO_SOT_Packages_SMD:SOT-23-5" H 6750 4200 50  0001 C CNN

Commit message: 2輪の基板を作成
部品を配置
Parts:
- removed R11: 10k, Resistors_SMD:R_0201, symbol R
- added C20: 0.1u, Capacitors_SMD:C_0201, symbol C_Small
- added P10, P7, P8, P9: Partition, symbol Partition
- D2: renamed from D3; symbol LED -> LED-RESCUE-KERISEv3
- R6: value 100 -> 47; footprint Resistors_SMD:R_0402 -> Resistors_SMD:R_0603
- U6: symbol MCP6001 -> MCP6001-RESCUE-KERISEv3
- renumbered C16 to C17, C15 to C18, C14 to C19, D2 to D3, P4 to P5, P5 to P6, R7 to R10, R10 to R7
Connections:
- net s_3.3V: now also C20.1
- net s_GND: now also C20.2
