File: kicad/esp32/Power.sch (KiCad schematic (older format))
At the start: 9 parts, among them P4 Battery, U5 NJM2884

Commit message: 自動配線成功
Parts:
- renumbered C16 to C11, C17 to C12, C18 to C13, P4 to P3
Changed lines of the file:
@@
 $Descr A4 11693 8268
 encoding utf-8
-Sheet 3 13
+Sheet 3 14
 Title ""
 Date ""
@@
 $EndDescr
 $Comp
-L +BATT #PWR023
+L +BATT #PWR020
 U 1 1 57CC111A
 P 2000 4200
-F 0 "#PWR023" H 2000 4050 50  0001 C CNN
+F 0 "#PWR020" H 2000 4050 50  0001 C CNN
 F 1 "+BATT" H 2000 4340 50  0000 C CNN
 F 2 "" H 2000 4200 50  0000 C CNN
@@
 $EndComp
 $Comp
-L GND #PWR024
+L GND #PWR021
 U 1 1 57CC113A
 P 2000 5200
-F 0 "#PWR024" H 2000 4950 50  0001 C CNN
+F 0 "#PWR021" H 2000 4950 50  0001 C CNN
 F 1 "GND" H 2000 5050 50  0000 C CNN
 F 2 "" H 2000 5200 50  0000 C CNN
@@
 $EndComp
 $Comp
-L GND #PWR025
+L GND #PWR022
 U 1 1 57CD3C05
 P 2700 5200
-F 0 "#PWR025" H 2700 4950 50  0001 C CNN
+F 0 "#PWR022" H 2700 4950 50  0001 C CNN
 F 1 "GND" H 2700 5050 50  0000 C CNN
 F 2 "" H 2700 5200 50  0000 C CNN
@@
 BAT_VOL
 $Comp
-L GND #PWR026
+L GND #PWR023
 U 1 1 57D18DB8
 P 2300 5200
-F 0 "#PWR026" H 2300 4950 50  0001 C CNN
+F 0 "#PWR023" H 2300 4950 50  0001 C CNN
 F 1 "GND" H 2300 5050 50  0000 C CNN
 F 2 "" H 2300 5200 50  0000 C CNN
@@
 $EndComp
 $Comp
-L PWR_FLAG #FLG027
+L PWR_FLAG #FLG024
 U 1 1 57D18DE7
 P 2300 5100
-F 0 "#FLG027" H 2300 5195 50  0001 C CNN
+F 0 "#FLG024" H 2300 5195 50  0001 C CNN
 F 1 "PWR_FLAG" H 2300 5280 50  0000 C CNN
 F 2 "" H 2300 5100 50  0000 C CNN
@@
 $EndComp
 $Comp
-L PWR_FLAG #FLG028
+L PWR_FLAG #FLG025
 U 1 1 57D1915C
 P 2300 4300
-F 0 "#FLG028" H 2300 4395 50  0001 C CNN
+F 0 "#FLG025" H 2300 4395 50  0001 C CNN
 F 1 "PWR_FLAG" H 2300 4480 50  0000 C CNN
 F 2 "" H 2300 4300 50  0000 C CNN
@@
 $EndComp
 $Comp
-L +BATT #PWR029
+L +BATT #PWR026
 U 1 1 57D1923B
 P 2300 4200
-F 0 "#PWR029" H 2300 4050 50  0001 C CNN
+F 0 "#PWR026" H 2300 4050 50  0001 C CNN
 F 1 "+BATT" H 2300 4340 50  0000 C CNN
 F 2 "" H 2300 4200 50  0000 C CNN
@@
 $EndComp
 $Comp
-L GND #PWR030
+L GND #PWR027
 U 1 1 57D00A42
 P 5900 5200
-F 0 "#PWR030" H 5900 4950 50  0001 C CNN
+F 0 "#PWR027" H 5900 4950 50  0001 C CNN
 F 1 "GND" H 5900 5050 50  0000 C CNN
 F 2 "" H 5900 5200 50  0000 C CNN
@@
 $EndComp
 $Comp
-L CONN_01X02 P4
+L CONN_01X02 P3
 U 1 1 57D07AC8
 P 1700 4450
-F 0 "P4" H 1700 4600 50  0000 C CNN
+F 0 "P3" H 1700 4600 50  0000 C CNN
 F 1 "Battery" V 1800 4450 50  0000 C CNN
 F 2 "Connectors_Hirose:Hirose_DF13-02P-1.25DSA_02x1.25mm_Straight" H 1700 4450 50  0001 C CNN
@@
 $EndComp
 $Comp
-L +BATT #PWR031
+L +BATT #PWR028
 U 1 1 589A7DD8
 P 3500 4200
-F 0 "#PWR031" H 3500 4050 50  0001 C CNN
+F 0 "#PWR028" H 3500 4050 50  0001 C CNN
 F 1 "+BATT" H 3500 4340 50  0000 C CNN
 F 2 "" H 3500 4200 50  0000 C CNN
@@
 $EndComp
 $Comp
-L C C16
+L C C11
 U 1 1 589A7E10
 P 3500 4850
-F 0 "C16" H 3525 4950 50  0000 L CNN
+F 0 "C11" H 3525 4950 50  0000 L CNN
 F 1 "0.33u" H 3525 4750 50  0000 L CNN
 F 2 "Capacitors_SMD:C_0201" H 3538 4700 50  0001 C CNN
@@
 $EndComp
 $Comp
-L GND #PWR032
+L GND #PWR029
 U 1 1 589A7FC5
 P 3500 5200
-F 0 "#PWR032" H 3500 4950 50  0001 C CNN
+F 0 "#PWR029" H 3500 4950 50  0001 C CNN
 F 1 "GND" H 3500 5050 50  0000 C CNN
 F 2 "" H 3500 5200 50  0000 C CNN
@@
 $EndComp
 $Comp
-L C C17
+L C C12
 U 1 1 589A830F
 P 5200 4850
-F 0 "C17" H 5225 4950 50  0000 L CNN
+F 0 "C12" H 5225 4950 50  0000 L CNN
 F 1 "0.1u" H 5225 4750 50  0000 L CNN
 F 2 "Capacitors_SMD:C_0201" H 5238 4700 50  0001 C CNN
@@
 $EndComp
 $Comp
-L GND #PWR033
+L GND #PWR030
 U 1 1 589A83D2
 P 5200 5200
-F 0 "#PWR033" H 5200 4950 50  0001 C CNN
+F 0 "#PWR030" H 5200 4950 50  0001 C CNN
 F 1 "GND" H 5200 5050 50  0000 C CNN
 F 2 "" H 5200 5200 50  0000 C CNN
@@
 $EndComp
 $Comp
-L +BATT #PWR034
+L +BATT #PWR031
 U 1 1 57CD3CA2
 P 2700 4200
-F 0 "#PWR034" H 2700 4050 50  0001 C CNN
+F 0 "#PWR031" H 2700 4050 50  0001 C CNN
 F 1 "+BATT" H 2700 4340 50  0000 C CNN
 F 2 "" H 2700 4200 50  0000 C CNN
@@
 $EndComp
 $Comp
-L GND #PWR035
+L GND #PWR032
 U 1 1 589A88D7
 P 5500 5200
-F 0 "#PWR035" H 5500 4950 50  0001 C CNN
+F 0 "#PWR032" H 5500 4950 50  0001 C CNN
 F 1 "GND" H 5500 5050 50  0000 C CNN
 F 2 "" H 5500 5200 50  0000 C CNN
@@
 $EndComp
 $Comp
-L C C18
+L C C13
 U 1 1 589A8858
 P 5500 4850
-F 0 "C18" H 5525 4950 50  0000 L CNN
+F 0 "C13" H 5525 4950 50  0000 L CNN
 F 1 "4.7u" H 5525 4750 50  0000 L CNN
 F 2 "Capacitors_SMD:C_0402" H 5538 4700 50  0001 C CNN
@@
 $EndComp
 $Comp
-L GND #PWR036
+L GND #PWR033
 U 1 1 589F7F11
 P 4900 5200
-F 0 "#PWR036" H 4900 4950 50  0001 C CNN
+F 0 "#PWR033" H 4900 4950 50  0001 C CNN
 F 1 "GND" H 4900 5050 50  0000 C CNN
 F 2 "" H 4900 5200 50  0000 C CNN
@@
 	1    0    0    -1
 $EndComp
-Connection ~ 3700 4300
-Wire Wire Line
-	3700 4400 3700 4300
-Wire Wire Line
-	3800 4400 3700 4400
-Wire Wire Line
-	4900 4500 4900 5200
-Wire Wire Line
-	2700 5100 2700 5200
-Wire Wire Line
-	2700 4200 2700 4300
-Wire Wire Line
-	2800 4700 2700 4700
-Wire Wire Line
-	2700 4600 2700 4800
-Connection ~ 2700 4700
-Wire Wire Line
-	2300 5100 2300 5200
-Wire Wire Line
-	2300 4200 2300 4300
-Wire Wire Line
-	5900 5200 5900 5100
-Wire Wire Line
-	5900 4700 5900 4600
-Wire Wire Line
-	5900 4300 5900 4200
-Wire Wire Line
-	1900 4500 2000 4500
-Wire Wire Line
-	2000 4500 2000 5200
-Wire Wire Line
-	3500 4200 3500 4700
-Connection ~ 3500 4300
-Wire Wire Line
-	3500 5000 3500 5200
-Connection ~ 5200 4300
-Wire Wire Line
-	5200 5000 5200 5200
-Wire Wire Line
-	5200 4300 5200 4700
-Wire Wire Line
-	3500 4300 3800 4300
-Connection ~ 5500 4300
-Wire Wire Line
-	4800 4300 5500 4300
-Wire Wire Line
-	5500 4200 5500 4700
-Wire Wire Line
-	5500 5000 5500 5200
-$Comp
-L +3.3V #PWR037
+$Comp
+L +3.3V #PWR034
 U 1 1 589CB5D5
 P 5500 4200
-F 0 "#PWR037" H 5500 4050 50  0001 C CNN
+F 0 "#PWR034" H 5500 4050 50  0001 C CNN
 F 1 "+3.3V" H 5500 4340 50  0000 C CNN
 F 2 "" H 5500 4200 50  0000 C CNN
@@
 $EndComp
 $Comp
-L +3.3V #PWR038
+L +3.3V #PWR035
 U 1 1 589CB64F
 P 5900 4200
-F 0 "#PWR038" H 5900 4050 50  0001 C CNN
+F 0 "#PWR035" H 5900 4050 50  0001 C CNN
 F 1 "+3.3V" H 5900 4340 50  0000 C CNN
 F 2 "" H 5900 4200 50  0000 C CNN
@@
 	1    0    0    -1
 $EndComp
+Connection ~ 3700 4300
+Wire Wire Line
+	3700 4400 3700 4300
+Wire Wire Line
+	3800 4400 3700 4400
+Wire Wire Line
+	4900 4500 4900 5200
+Wire Wire Line
+	2700 5100 2700 5200
+Wire Wire Line
+	2700 4200 2700 4300
+Wire Wire Line
+	2800 4700 2700 4700
+Wire Wire Line
+	2700 4600 2700 4800
+Connection ~ 2700 4700
+Wire Wire Line
+	2300 5100 2300 5200
+Wire Wire Line
+	2300 4200 2300 4300
+Wire Wire Line
+	5900 5200 5900 5100
+Wire Wire Line
+	5900 4700 5900 4600
+Wire Wire Line
+	5900 4300 5900 4200
+Wire Wire Line
+	1900 4500 2000 4500
+Wire Wire Line
+	2000 4500 2000 5200
+Wire Wire Line
+	3500 4200 3500 4700
+Connection ~ 3500 4300
+Wire Wire Line
+	3500 5000 3500 5200
+Connection ~ 5200 4300
+Wire Wire Line
+	5200 5000 5200 5200
+Wire Wire Line
+	5200 4300 5200 4700
+Wire Wire Line
+	3500 4300 3800 4300
+Connection ~ 5500 4300
+Wire Wire Line
+	4800 4300 5500 4300
+Wire Wire Line
+	5500 4200 5500 4700
+Wire Wire Line
+	5500 5000 5500 5200
 Wire Wire Line
 	2000 4200 2000 4400
 Wire Wire Line
 	2000 4400 1900 4400
+Wire Wire Line
+	4900 4500 4800 4500
 $Comp
 L NJM2884 U5
@@
 	1    0    0    -1
 $EndComp
-Wire Wire Line
-	4900 4500 4800 4500
 $EndSCHEMATC

Commit message: 2輪の基板を作成
部品を配置
Parts:
- removed C11: 0.33u, Capacitors_SMD:C_0201, symbol C
- removed C12: 0.1u, Capacitors_SMD:C_0201, symbol C
- removed C13: 4.7u, Capacitors_SMD:C_0402, symbol C
- removed U5: NJM2884, TO_SOT_Packages_SMD:SOT89-5_Housing, symbol NJM2884
- added C15: 10u, Capacitors_SMD:C_0603, symbol C_Small
- added C16: 47u, Capacitors_SMD:C_0805, symbol C_Small
- added U5: LXDC2URxx, mouse:LXDC2UR, symbol LXDC2URxx
- D1: symbol LED -> LED-RESCUE-KERISEv3
- renumbered P3 to P4, R5 to R4, R4 to R5
Connections:
- net +3V3: now also C16.1, U5.3 (Vout), U5.4 (Vout)
- net +BATT: now also C15.1, U5.5 (EN), U5.7 (Vin), U5.8 (Vin)
- net GND: now also C15.2, C16.2, U5.2 (GND), U5.6 (GND), U5.9 (GND)
- no-connect marks 0 -> 1
Other:
- moved on the sheet: D1, R5
