File: kicad/esp32/UI.sch (KiCad schematic (older format))
At the start: 10 parts, among them Q5 BSS138, SW2 SW_PUSH_SMALL

Commit message: 更新
Parts:
- removed D12: LED, LEDs:LED_0402, symbol LED
- removed R32: 1k, Resistors_SMD:R_0201, symbol R
- renumbered R33 to R32
Other:
- moved on the sheet: SW2
Changed lines of the file:
@@
 $EndComp
 $Comp
-L R R33
+L R R32
 U 1 1 57CE757A
 P 4000 4450
-F 0 "R33" V 4080 4450 50  0000 C CNN
+F 0 "R32" V 4080 4450 50  0000 C CNN
 F 1 "10k" V 4000 4450 50  0000 C CNN
 F 2 "Resistors_SMD:R_0201" V 3930 4450 50  0001 C CNN
@@
 $EndComp
 $Comp
-L LED D12
-U 1 1 57CE815D
-P 6300 4400
-F 0 "D12" H 6300 4500 50  0000 C CNN
-F 1 "LED" H 6300 4300 50  0000 C CNN
-F 2 "LEDs:LED_0402" H 6300 4400 50  0001 C CNN
-F 3 "" H 6300 4400 50  0000 C CNN
-	1    6300 4400
-	0    -1   -1   0
-$EndComp
-$Comp
 L GND #PWR051
 U 1 1 57CE8530
@@
 	1    0    0    -1
 $EndComp
-$Comp
-L GND #PWR053
-U 1 1 57CE8577
-P 6300 4700
-F 0 "#PWR053" H 6300 4450 50  0001 C CNN
-F 1 "GND" H 6300 4550 50  0000 C CNN
-F 2 "" H 6300 4700 50  0000 C CNN
-F 3 "" H 6300 4700 50  0000 C CNN
-	1    6300 4700
-	1    0    0    -1
-$EndComp
-Wire Wire Line
-	6300 4600 6300 4700
 Wire Wire Line
 	6000 4700 6000 4600
@@
 	1    0    0    -1
 $EndComp
-$Comp
-L R R32
-U 1 1 57CE8677
-P 6300 3950
-F 0 "R32" V 6380 3950 50  0000 C CNN
-F 1 "1k" V 6300 3950 50  0000 C CNN
-F 2 "Resistors_SMD:R_0201" V 6230 3950 50  0001 C CNN
-F 3 "" H 6300 3950 50  0000 C CNN
-	1    6300 3950
-	1    0    0    -1
-$EndComp
-Wire Wire Line
-	6300 4200 6300 4100
 Wire Wire Line
 	6000 4100 6000 4200
@@
 Text HLabel 5600 3600 0    60   Input ~ 0
 LED_2
-Text HLabel 5600 3500 0    60   Input ~ 0
-LED_3
 Wire Wire Line
 	5600 3700 5700 3700
@@
 Wire Wire Line
 	6000 3600 6000 3800
-Wire Wire Line
-	6300 3800 6300 3500
-Wire Wire Line
-	6300 3500 5600 3500
 $Comp
-L GND #PWR054
+L GND #PWR053
 U 1 1 57CEA2EF
-P 7200 4700
-F 0 "#PWR054" H 7200 4450 50  0001 C CNN
-F 1 "GND" H 7200 4550 50  0000 C CNN
-F 2 "" H 7200 4700 50  0000 C CNN
-F 3 "" H 7200 4700 50  0000 C CNN
-	1    7200 4700
+P 6900 4700
+F 0 "#PWR053" H 6900 4450 50  0001 C CNN
+F 1 "GND" H 6900 4550 50  0000 C CNN
+F 2 "" H 6900 4700 50  0000 C CNN
+F 3 "" H 6900 4700 50  0000 C CNN
+	1    6900 4700
 	1    0    0    -1
 $EndComp
 Wire Wire Line
-	7200 4700 7200 4500
-Text HLabel 7000 3800 0    60   Input ~ 0
+	6900 4700 6900 4500
+Text HLabel 6700 3800 0    60   Input ~ 0
 BUTTON
 Text Notes 3300 3100 0    100  ~ 0
@@
 L SW_PUSH_SMALL SW2
 U 1 1 589B56D0
-P 7100 4400
-F 0 "SW2" H 7250 4510 50  0000 C CNN
-F 1 "SW_PUSH_SMALL" H 7100 4321 50  0000 C CNN
-F 2 "Buttons_Switches_SMD:SW_SPST_KMR2" H 7100 4400 50  0001 C CNN
-F 3 "" H 7100 4400 50  0000 C CNN
-	1    7100 4400
+P 6800 4400
+F 0 "SW2" H 6950 4510 50  0000 C CNN
+F 1 "SW_PUSH_SMALL" H 6800 4321 50  0000 C CNN
+F 2 "Buttons_Switches_SMD:SW_SPST_KMR2" H 6800 4400 50  0001 C CNN
+F 3 "" H 6800 4400 50  0000 C CNN
+	1    6800 4400
 	1    0    0    -1
 $EndComp
 Wire Wire Line
-	7000 3800 7000 4300
+	6700 3800 6700 4300
 $Comp
-L +3.3V #PWR055
+L +3.3V #PWR054
 U 1 1 589CB988
 P 4400 3500
-F 0 "#PWR055" H 4400 3350 50  0001 C CNN
+F 0 "#PWR054" H 4400 3350 50  0001 C CNN
 F 1 "+3.3V" H 4400 3640 50  0000 C CNN
 F 2 "" H 4400 3500 50  0000 C CNN

Commit message: 2輪の基板を作成
部品を配置
Parts:
- removed R32: 10k, Resistors_SMD:R_0201, symbol R
- added C25: 0.1u, Capacitors_SMD:C_0201, symbol C_Small
- added D8: LED, LEDs:LED_0402, symbol LED-RESCUE-KERISEv3
- added R16: 1k, Resistors_SMD:R_0201, symbol R_Small
- added R19: 1k, Resistors_SMD:R_0201, symbol R
- D6: renamed from D10; symbol LED -> LED-RESCUE-KERISEv3
- D7: renamed from D11; symbol LED -> LED-RESCUE-KERISEv3
- Q3: renamed from Q5; value BSS138 -> IRFML8244
- SW2: footprint Buttons_Switches_SMD:SW_SPST_KMR2 -> mouse:SW_PUSH
- renumbered R30 to R17, R31 to R18
Connections:
- net GND: now also D8.1 (K)
- net at SP1.2: now also R16.1; no longer Q3.3 (D)
- new net: C25.2, Q3.3 (D)
- new net: D8.2 (A), R19.2
- new net: C25.1, R16.2
- new net LED_3: R19.1
Other:
- moved on the sheet: SP1, SW2
Changed lines of the file:
@@
 $Descr A4 11693 8268
 encoding utf-8
-Sheet 9 14
+Sheet 6 13
 Title ""
 Date ""
@@
 L SPEAKER SP1
 U 1 1 57CD8DE7
-P 4800 3700
-F 0 "SP1" H 4700 3950 50  0000 C CNN
-F 1 "SMT-0440" H 4700 3450 50  0000 C CNN
-F 2 "mouse:SMT-0440-S-R" H 4800 3700 50  0001 C CNN
-F 3 "" H 4800 3700 50  0000 C CNN
-	1    4800 3700
-	1    0    0    -1
-$EndComp
-$Comp
-L R R32
-U 1 1 57CE757A
-P 4000 4450
-F 0 "R32" V 4080 4450 50  0000 C CNN
-F 1 "10k" V 4000 4450 50  0000 C CNN
-F 2 "Resistors_SMD:R_0201" V 3930 4450 50  0001 C CNN
-F 3 "" H 4000 4450 50  0000 C CNN
-	1    4000 4450
-	1    0    0    -1
-$EndComp
-$Comp
-L Q_NMOS_GSD Q5
+P 4800 3200
+F 0 "SP1" H 4700 3450 50  0000 C CNN
+F 1 "SMT-0440" H 4850 3550 50  0000 C CNN
+F 2 "mouse:SMT-0440-S-R" H 4800 3200 50  0001 C CNN
+F 3 "" H 4800 3200 50  0000 C CNN
+	1    4800 3200
+	1    0    0    -1
+$EndComp
+$Comp
+L Q_NMOS_GSD Q3
 U 1 1 57CE75AD
 P 4300 4200
-F 0 "Q5" H 4600 4250 50  0000 R CNN
-F 1 "BSS138" H 4800 4150 50  0000 R CNN
+F 0 "Q3" H 4600 4250 50  0000 R CNN
+F 1 "IRFML8244" H 4350 4400 50  0000 R CNN
 F 2 "TO_SOT_Packages_SMD:SOT-23" H 4500 4300 50  0001 C CNN
 F 3 "" H 4300 4200 50  0000 C CNN
@@
 $EndComp
 $Comp
-L GND #PWR049
+L GND #PWR042
 U 1 1 57CE7673
 P 4400 4700
-F 0 "#PWR049" H 4400 4450 50  0001 C CNN
+F 0 "#PWR042" H 4400 4450 50  0001 C CNN
 F 1 "GND" H 4400 4550 50  0000 C CNN
 F 2 "" H 4400 4700 50  0000 C CNN
@@
 	1    0    0    -1
 $EndComp
-$Comp
-L GND #PWR050
-U 1 1 57CE768B
-P 4000 4700
-F 0 "#PWR050" H 4000 4450 50  0001 C CNN
-F 1 "GND" H 4000 4550 50  0000 C CNN
-F 2 "" H 4000 4700 50  0000 C CNN
-F 3 "" H 4000 4700 50  0000 C CNN
-	1    4000 4700
-	1    0    0    -1
-$EndComp
 Text HLabel 3900 4200 0    60   Input ~ 0
 SPEAKER
 Wire Wire Line
-	4400 3500 4400 3600
-Wire Wire Line
-	4400 3600 4500 3600
-Wire Wire Line
-	4500 3800 4400 3800
-Wire Wire Line
-	4400 3800 4400 4000
+	4400 3000 4400 3100
+Wire Wire Line
+	4400 3100 4500 3100
+Wire Wire Line
+	4500 3300 4400 3300
 Wire Wire Line
 	4400 4400 4400 4700
 Wire Wire Line
 	3900 4200 4100 4200
-Wire Wire Line
-	4000 4200 4000 4300
-Wire Wire Line
-	4000 4700 4000 4600
-Connection ~ 4000 4200
-$Comp
-L LED D10
+$Comp
+L LED-RESCUE-KERISEv3 D6
 U 1 1 57CE80D9
 P 5700 4400
-F 0 "D10" H 5700 4500 50  0000 C CNN
+F 0 "D6" H 5700 4500 50  0000 C CNN
 F 1 "LED" H 5700 4300 50  0000 C CNN
 F 2 "LEDs:LED_0402" H 5700 4400 50  0001 C CNN
@@
 $EndComp
 $Comp
-L LED D11
+L LED-RESCUE-KERISEv3 D7
 U 1 1 57CE812A
 P 6000 4400
-F 0 "D11" H 6000 4500 50  0000 C CNN
+F 0 "D7" H 6000 4500 50  0000 C CNN
 F 1 "LED" H 6000 4300 50  0000 C CNN
 F 2 "LEDs:LED_0402" H 6000 4400 50  0001 C CNN
@@
 $EndComp
 $Comp
-L GND #PWR051
+L GND #PWR043
 U 1 1 57CE8530
 P 5700 4700
-F 0 "#PWR051" H 5700 4450 50  0001 C CNN
+F 0 "#PWR043" H 5700 4450 50  0001 C CNN
 F 1 "GND" H 5700 4550 50  0000 C CNN
 F 2 "" H 5700 4700 50  0000 C CNN
@@
 $EndComp
 $Comp
-L GND #PWR052
+L GND #PWR044
 U 1 1 57CE8557
 P 6000 4700
-F 0 "#PWR052" H 6000 4450 50  0001 C CNN
+F 0 "#PWR044" H 6000 4450 50  0001 C CNN
 F 1 "GND" H 6000 4550 50  0000 C CNN
 F 2 "" H 6000 4700 50  0000 C CNN
@@
 	5700 4600 5700 4700
 $Comp
-L R R30
+L R R17
 U 1 1 57CE8600
 P 5700 3950
-F 0 "R30" V 5780 3950 50  0000 C CNN
+F 0 "R17" V 5780 3950 50  0000 C CNN
 F 1 "1k" V 5700 3950 50  0000 C CNN
 F 2 "Resistors_SMD:R_0201" V 5630 3950 50  0001 C CNN
@@
 $EndComp
 $Comp
-L R R31
+L R R18
 U 1 1 57CE8644
 P 6000 3950
-F 0 "R31" V 6080 3950 50  0000 C CNN
+F 0 "R18" V 6080 3950 50  0000 C CNN
 F 1 "1k" V 6000 3950 50  0000 C CNN
 F 2 "Resistors_SMD:R_0201" V 5930 3950 50  0001 C CNN
@@
 	6000 3600 6000 3800
 $Comp
-L GND #PWR053
+L GND #PWR045
 U 1 1 57CEA2EF
-P 6900 4700
-F 0 "#PWR053" H 6900 4450 50  0001 C CNN
-F 1 "GND" H 6900 4550 50  0000 C CNN
-F 2 "" H 6900 4700 50  0000 C CNN
-F 3 "" H 6900 4700 50  0000 C CNN
-	1    6900 4700
-	1    0    0    -1
-$EndComp
-Wire Wire Line
-	6900 4700 6900 4500
-Text HLabel 6700 3800 0    60   Input ~ 0
+P 7200 4700
+F 0 "#PWR045" H 7200 4450 50  0001 C CNN
+F 1 "GND" H 7200 4550 50  0000 C CNN
+F 2 "" H 7200 4700 50  0000 C CNN
+F 3 "" H 7200 4700 50  0000 C CNN
+	1    7200 4700
+	1    0    0    -1
+$EndComp
+Wire Wire Line
+	7200 4700 7200 4500
+Text HLabel 7000 3800 0    60   Input ~ 0
 BUTTON
-Text Notes 3300 3100 0    100  ~ 0
+Text Notes 3300 2700 0    100  ~ 0
 User Interface
 $Comp
 L SW_PUSH_SMALL SW2
 U 1 1 589B56D0
-P 6800 4400
-F 0 "SW2" H 6950 4510 50  0000 C CNN
-F 1 "SW_PUSH_SMALL" H 6800 4321 50  0000 C CNN
-F 2 "Buttons_Switches_SMD:SW_SPST_KMR2" H 6800 4400 50  0001 C CNN
-F 3 "" H 6800 4400 50  0000 C CNN
-	1    6800 4400
-	1    0    0    -1
-$EndComp
-Wire Wire Line
-	6700 3800 6700 4300
-$Comp
-L +3.3V #PWR054
+P 7100 4400
+F 0 "SW2" H 7250 4510 50  0000 C CNN
+F 1 "SW_PUSH_SMALL" H 7100 4321 50  0000 C CNN
+F 2 "mouse:SW_PUSH" H 7100 4400 50  0001 C CNN
+F 3 "" H 7100 4400 50  0000 C CNN
+	1    7100 4400
+	1    0    0    -1
+$EndComp
+Wire Wire Line
+	7000 3800 7000 4300
+$Comp
+L +3.3V #PWR046
 U 1 1 589CB988
+P 4400 3000
+F 0 "#PWR046" H 4400 2850 50  0001 C CNN
+F 1 "+3.3V" H 4400 3140 50  0000 C CNN
+F 2 "" H 4400 3000 50  0000 C CNN
+F 3 "" H 4400 3000 50  0000 C CNN
+	1    4400 3000
+	1    0    0    -1
+$EndComp
+$Comp
+L LED-RESCUE-KERISEv3 D8
+U 1 1 592C69B3
+P 6300 4400
+F 0 "D8" H 6300 4500 50  0000 C CNN
+F 1 "LED" H 6300 4300 50  0000 C CNN
+F 2 "LEDs:LED_0402" H 6300 4400 50  0001 C CNN
+F 3 "" H 6300 4400 50  0000 C CNN
+	1    6300 4400
+	0    -1   -1   0
+$EndComp
+$Comp
+L GND #PWR047
+U 1 1 592C69B9
+P 6300 4700
+F 0 "#PWR047" H 6300 4450 50  0001 C CNN
+F 1 "GND" H 6300 4550 50  0000 C CNN
+F 2 "" H 6300 4700 50  0000 C CNN
+F 3 "" H 6300 4700 50  0000 C CNN
+	1    6300 4700
+	1    0    0    -1
+$EndComp
+Wire Wire Line
+	6300 4700 6300 4600
+$Comp
+L R R19
+U 1 1 592C69C0
+P 6300 3950
+F 0 "R19" V 6380 3950 50  0000 C CNN
+F 1 "1k" V 6300 3950 50  0000 C CNN
+F 2 "Resistors_SMD:R_0201" V 6230 3950 50  0001 C CNN
+F 3 "" H 6300 3950 50  0000 C CNN
+	1    6300 3950
+	1    0    0    -1
+$EndComp
+Wire Wire Line
+	6300 4100 6300 4200
+Wire Wire Line
+	6300 3500 6300 3800
+Text HLabel 5600 3500 0    60   Input ~ 0
+LED_3
+Wire Wire Line
+	5600 3500 6300 3500
+$Comp
+L C_Small C25
+U 1 1 594481A2
+P 4400 3800
+F 0 "C25" H 4410 3870 50  0000 L CNN
+F 1 "0.1u" H 4410 3720 50  0000 L CNN
+F 2 "Capacitors_SMD:C_0201" H 4400 3800 50  0001 C CNN
+F 3 "" H 4400 3800 50  0001 C CNN
+	1    4400 3800
+	1    0    0    -1
+$EndComp
+Wire Wire Line
+	4400 3300 4400 3400
+Wire Wire Line
+	4400 3600 4400 3700
+$Comp
+L R_Small R16
+U 1 1 5945E920
 P 4400 3500
-F 0 "#PWR054" H 4400 3350 50  0001 C CNN
-F 1 "+3.3V" H 4400 3640 50  0000 C CNN
-F 2 "" H 4400 3500 50  0000 C CNN
-F 3 "" H 4400 3500 50  0000 C CNN
+F 0 "R16" H 4430 3520 50  0000 L CNN
+F 1 "1k" H 4430 3460 50  0000 L CNN
+F 2 "Resistors_SMD:R_0201" H 4400 3500 50  0001 C CNN
+F 3 "" H 4400 3500 50  0001 C CNN
 	1    4400 3500
 	1    0    0    -1
 $EndComp
+Wire Wire Line
+	4400 4000 4400 3900
 $EndSCHEMATC
