File: kicad/AXIS_SENSOR.sch (KiCad schematic (older format))
At the start: 3 parts, among them U13 ICM-20602

Commit message: 4輪の改良版を設計
Parts:
- renumbered C34 to C30, C35 to C31, U13 to U11
Changed lines of the file:
@@
 LIBS:zetex
 LIBS:Zilog
-LIBS:KERISE-cache
 EELAYER 25 0
 EELAYER END
 $Descr A4 11693 8268
 encoding utf-8
-Sheet 13 13
+Sheet 13 14
 Title ""
 Date ""
@@
 AXIS Sensor
 $Comp
-L ICM-20602 U13
+L ICM-20602 U11
 U 1 1 592C611A
 P 5600 3400
-F 0 "U13" H 5600 4150 60  0000 C CNN
+F 0 "U11" H 5600 4150 60  0000 C CNN
 F 1 "ICM-20602" H 5600 4000 60  0000 C CNN
 F 2 "mouse:LGA-16-3x3" H 5600 4000 60  0001 C CNN
@@
 $EndComp
 $Comp
-L C_Small C35
+L C_Small C31
 U 1 1 592C613A
 P 4800 3700
-F 0 "C35" H 4810 3770 50  0000 L CNN
+F 0 "C31" H 4810 3770 50  0000 L CNN
 F 1 "0.1u" H 4810 3620 50  0000 L CNN
 F 2 "Capacitors_SMD:C_0201" H 4800 3700 50  0001 C CNN
@@
 $EndComp
 $Comp
-L C_Small C34
+L C_Small C30
 U 1 1 592C6186
 P 4600 3700
-F 0 "C34" H 4610 3770 50  0000 L CNN
+F 0 "C30" H 4610 3770 50  0000 L CNN
 F 1 "0.1u" H 4610 3620 50  0000 L CNN
 F 2 "Capacitors_SMD:C_0201" H 4600 3700 50  0001 C CNN
@@
 $EndComp
 $Comp
-L GND #PWR072
+L GND #PWR069
 U 1 1 592C63E1
 P 5000 4200
-F 0 "#PWR072" H 5000 3950 50  0001 C CNN
+F 0 "#PWR069" H 5000 3950 50  0001 C CNN
 F 1 "GND" H 5000 4050 50  0000 C CNN
 F 2 "" H 5000 4200 50  0000 C CNN
@@
 $EndComp
 $Comp
-L GND #PWR073
+L GND #PWR070
 U 1 1 592C640D
 P 4800 4200
-F 0 "#PWR073" H 4800 3950 50  0001 C CNN
+F 0 "#PWR070" H 4800 3950 50  0001 C CNN
 F 1 "GND" H 4800 4050 50  0000 C CNN
 F 2 "" H 4800 4200 50  0000 C CNN
@@
 $EndComp
 $Comp
-L GND #PWR074
+L GND #PWR071
 U 1 1 592C6444
 P 4600 4200
-F 0 "#PWR074" H 4600 3950 50  0001 C CNN
+F 0 "#PWR071" H 4600 3950 50  0001 C CNN
 F 1 "GND" H 4600 4050 50  0000 C CNN
 F 2 "" H 4600 4200 50  0000 C CNN
@@
 $EndComp
 $Comp
-L +3.3V #PWR075
+L +3.3V #PWR072
 U 1 1 592C64FB
 P 5000 2800
-F 0 "#PWR075" H 5000 2650 50  0001 C CNN
+F 0 "#PWR072" H 5000 2650 50  0001 C CNN
 F 1 "+3.3V" H 5000 2940 50  0000 C CNN
 F 2 "" H 5000 2800 50  0000 C CNN
@@
 NoConn ~ 6100 3300
 $Comp
-L GND #PWR076
+L GND #PWR073
 U 1 1 592C6B85
 P 6200 3500
-F 0 "#PWR076" H 6200 3250 50  0001 C CNN
+F 0 "#PWR073" H 6200 3250 50  0001 C CNN
 F 1 "GND" H 6200 3350 50  0000 C CNN
 F 2 "" H 6200 3500 50  0000 C CNN
