File: kicad/AXIS_SENSOR.sch (KiCad schematic (older format))
At the start: 3 parts, among them U11 ICM-20602

Commit message: 回路とフットプリントを改良
Parts:
- renumbered C30 to C32, C31 to C33
Changed lines of the file:
@@
 $EndComp
 $Comp
-L C_Small C31
+L C_Small C33
 U 1 1 592C613A
 P 4800 3700
-F 0 "C31" H 4810 3770 50  0000 L CNN
+F 0 "C33" H 4810 3770 50  0000 L CNN
 F 1 "0.1u" H 4810 3620 50  0000 L CNN
 F 2 "Capacitors_SMD:C_0201" H 4800 3700 50  0001 C CNN
@@
 $EndComp
 $Comp
-L C_Small C30
+L C_Small C32
 U 1 1 592C6186
 P 4600 3700
-F 0 "C30" H 4610 3770 50  0000 L CNN
+F 0 "C32" H 4610 3770 50  0000 L CNN
 F 1 "0.1u" H 4610 3620 50  0000 L CNN
 F 2 "Capacitors_SMD:C_0201" H 4600 3700 50  0001 C CNN
@@
 $EndComp
 $Comp
-L GND #PWR069
+L GND #PWR074
 U 1 1 592C63E1
 P 5000 4200
-F 0 "#PWR069" H 5000 3950 50  0001 C CNN
+F 0 "#PWR074" H 5000 3950 50  0001 C CNN
 F 1 "GND" H 5000 4050 50  0000 C CNN
 F 2 "" H 5000 4200 50  0000 C CNN
@@
 $EndComp
 $Comp
-L GND #PWR070
+L GND #PWR075
 U 1 1 592C640D
 P 4800 4200
-F 0 "#PWR070" H 4800 3950 50  0001 C CNN
+F 0 "#PWR075" H 4800 3950 50  0001 C CNN
 F 1 "GND" H 4800 4050 50  0000 C CNN
 F 2 "" H 4800 4200 50  0000 C CNN
@@
 $EndComp
 $Comp
-L GND #PWR071
+L GND #PWR076
 U 1 1 592C6444
 P 4600 4200
-F 0 "#PWR071" H 4600 3950 50  0001 C CNN
+F 0 "#PWR076" H 4600 3950 50  0001 C CNN
 F 1 "GND" H 4600 4050 50  0000 C CNN
 F 2 "" H 4600 4200 50  0000 C CNN
@@
 $EndComp
 $Comp
-L +3.3V #PWR072
+L +3.3V #PWR077
 U 1 1 592C64FB
 P 5000 2800
-F 0 "#PWR072" H 5000 2650 50  0001 C CNN
+F 0 "#PWR077" H 5000 2650 50  0001 C CNN
 F 1 "+3.3V" H 5000 2940 50  0000 C CNN
 F 2 "" H 5000 2800 50  0000 C CNN
@@
 NoConn ~ 6100 3300
 $Comp
-L GND #PWR073
+L GND #PWR078
 U 1 1 592C6B85
 P 6200 3500
-F 0 "#PWR073" H 6200 3250 50  0001 C CNN
+F 0 "#PWR078" H 6200 3250 50  0001 C CNN
 F 1 "GND" H 6200 3350 50  0000 C CNN
 F 2 "" H 6200 3500 50  0000 C CNN
