File: kicad/KERISE.sch (KiCad schematic (older format))
At the start: 20 parts, among them P1 ANT, SW1 SW_Push, U1 FLASH, U2 ESP32, U3 XTAL

Commit message: 3.3Vの電源ラインを強化，変換基板を付属
Parts:
- added U14: FLASH, Housings_DFN_QFN:DFN-8-1EP_3x2mm_Pitch0.5mm, symbol FLASH
- added U15: FLASH, mouse:SOIJ-8_5.3x5.3mm_Pitch1.27mm_th, symbol FLASH
- U1: footprint mouse:DFN-8-1EP_6x5mm_Pitch1.27mm_SmallFlag -> mouse:SOIJ-8_5.3x5.3mm_Pitch1.27mm
Connections:
- new net: U14.1 (~CS), U15.1 (~CS)
- new net: U14.2 (DO), U15.2 (DO)
- new net: U14.3 (~WP), U15.3 (~WP)
- new net: U14.4 (GND), U15.4 (GND)
- new net: U14.5 (DI), U15.5 (DI)
- new net: U14.6 (CLK), U15.6 (CLK)
- new net: U14.7 (~HOLD), U15.7 (~HOLD)
- new net: U14.8 (VCC), U15.8 (VCC)
Changed lines of the file:
@@
 F 0 "U1" H 5150 6250 60  0000 C CNN
 F 1 "FLASH" H 5200 6150 60  0000 C CNN
-F 2 "mouse:DFN-8-1EP_6x5mm_Pitch1.27mm_SmallFlag" H 5000 6050 60  0001 C CNN
+F 2 "mouse:SOIJ-8_5.3x5.3mm_Pitch1.27mm" H 5000 6050 60  0001 C CNN
 F 3 "" H 5000 6050 60  0000 C CNN
 	1    5000 6050
@@
 Wire Wire Line
 	8600 3400 8700 3400
+$Comp
+L FLASH U14
+U 1 1 596DBCAE
+P 6300 6850
+F 0 "U14" H 6450 7050 60  0000 C CNN
+F 1 "FLASH" H 6500 6950 60  0000 C CNN
+F 2 "Housings_DFN_QFN:DFN-8-1EP_3x2mm_Pitch0.5mm" H 6300 6850 60  0001 C CNN
+F 3 "" H 6300 6850 60  0000 C CNN
+	1    6300 6850
+	1    0    0    -1
+$EndComp
+$Comp
+L FLASH U15
+U 1 1 596DBDE5
+P 6300 6850
+F 0 "U15" H 6450 7050 60  0000 C CNN
+F 1 "FLASH" H 6500 6950 60  0000 C CNN
+F 2 "mouse:SOIJ-8_5.3x5.3mm_Pitch1.27mm_th" H 6300 6850 60  0001 C CNN
+F 3 "" H 6300 6850 60  0000 C CNN
+	1    6300 6850
+	1    0    0    -1
+$EndComp
 $EndSCHEMATC

Commit message: 4輪の改良版を設計
Parts:
- removed U14: FLASH, Housings_DFN_QFN:DFN-8-1EP_3x2mm_Pitch0.5mm, symbol FLASH
- removed U15: FLASH, mouse:SOIJ-8_5.3x5.3mm_Pitch1.27mm_th, symbol FLASH
Connections:
- net BAT-VOL: now also U2.11 (GPI35/VDET_2/ADC1_CH7); no longer U2.5 (GPI36/SENSOR_VP/ADC1_CH0)
- net PR-RCV-SR: now reaches U2.6 (GPI37/SENSOR_CAPP/ADC1_CH1)
- net PR-RCV-FL: now reaches U2.7 (GPI38/SENSOR_CAPN/ADC1_CH2)
- net PR-RCV-FR: now reaches U2.8 (GPI39/SENSOR_VN/ADC1_CH3)
- net PR-LED-L renamed PR-LED-SL
- net PR-LED-R renamed PR-LED-SR
- net PR-RCV-L: no longer names the net of U2.10 (GPI34/VDET_1/ADC1_CH6)
- net PR-RCV-R renamed LED_4
- new net PR-RCV-SL: U2.5 (GPI36/SENSOR_VP/ADC1_CH0)
- no-connect marks 4 -> 1
Other:
- moved on the sheet: C1, C10, C11, C12, C2, C3, C4, C5, C6, C7, C8, C9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
