File: kicad/UI.sch (KiCad schematic (older format))
At the start: 11 parts, among them Q3 IRFML8244, SW2 SW_Push

Commit message: 4輪の改良版を設計
Parts:
- added D9: LED, LEDs:LED_0402, symbol LED
- added R20: 1k, Resistors_SMD:R_0201, symbol R
- Q3: value IRFML8244 -> NX3020NAKW; footprint TO_SOT_Packages_SMD:SOT-23 -> TO_SOT_Packages_SMD:SOT-323_SC-70
Connections:
- net GND: now also D9.1 (K)
- new net: D9.2 (A), R20.2
- new net LED_4: R20.1
Changed lines of the file:
@@
 LIBS:zetex
 LIBS:Zilog
-LIBS:KERISE-cache
 EELAYER 25 0
 EELAYER END
 $Descr A4 11693 8268
 encoding utf-8
-Sheet 6 13
+Sheet 6 14
 Title ""
 Date ""
@@
 P 4300 4200
 F 0 "Q3" H 4600 4250 50  0000 R CNN
-F 1 "IRFML8244" H 4350 4400 50  0000 R CNN
-F 2 "TO_SOT_Packages_SMD:SOT-23" H 4500 4300 50  0001 C CNN
+F 1 "NX3020NAKW" H 4350 4400 50  0000 R CNN
+F 2 "TO_SOT_Packages_SMD:SOT-323_SC-70" H 4500 4300 50  0001 C CNN
 F 3 "" H 4300 4200 50  0000 C CNN
 	1    4300 4200
@@
 Wire Wire Line
 	7200 3800 7200 4100
+$Comp
+L GND #PWR052
+U 1 1 5980F69C
+P 6600 4700
+F 0 "#PWR052" H 6600 4450 50  0001 C CNN
+F 1 "GND" H 6600 4550 50  0000 C CNN
+F 2 "" H 6600 4700 50  0000 C CNN
+F 3 "" H 6600 4700 50  0000 C CNN
+	1    6600 4700
+	1    0    0    -1
+$EndComp
+Wire Wire Line
+	6600 4700 6600 4600
+$Comp
+L R R20
+U 1 1 5980F6A3
+P 6600 4050
+F 0 "R20" V 6680 4050 50  0000 C CNN
+F 1 "1k" V 6600 4050 50  0000 C CNN
+F 2 "Resistors_SMD:R_0201" V 6530 4050 50  0001 C CNN
+F 3 "" H 6600 4050 50  0000 C CNN
+	1    6600 4050
+	1    0    0    -1
+$EndComp
+Wire Wire Line
+	6600 4200 6600 4300
+Wire Wire Line
+	6600 3500 6600 3900
+$Comp
+L LED D9
+U 1 1 5980F6AC
+P 6600 4450
+F 0 "D9" H 6600 4550 50  0000 C CNN
+F 1 "LED" H 6600 4350 50  0000 C CNN
+F 2 "LEDs:LED_0402" H 6600 4450 50  0001 C CNN
+F 3 "" H 6600 4450 50  0001 C CNN
+	1    6600 4450
+	0    -1   -1   0
+$EndComp
+Text HLabel 5600 3500 0    60   Input ~ 0
+LED_4
+Wire Wire Line
+	5600 3500 6600 3500
 $EndSCHEMATC
