File: kicad/Writer.sch (KiCad schematic (older format))
At the start: 12 parts, among them J1 USB_OTG, P23 COM, U10 MCP73831, U11 FT234XD

Commit message: 自動配線成功
Parts:
- U11: footprint Housings_DFN_QFN:DFN-12-1EP_3x3mm_Pitch0.45mm -> mouse:DFN-12-1EP_3x3mm_Pitch0.45mm
Changed lines of the file:
@@
 F 0 "U11" H 6100 4250 60  0000 C CNN
 F 1 "FT234XD" H 6100 4100 60  0000 C CNN
-F 2 "Housings_DFN_QFN:DFN-12-1EP_3x3mm_Pitch0.45mm" H 6100 4100 60  0001 C CNN
+F 2 "mouse:DFN-12-1EP_3x3mm_Pitch0.45mm" H 6100 4100 60  0001 C CNN
 F 3 "" H 6100 4100 60  0000 C CNN
 	1    6100 3700

Commit message: 4輪の改良版を設計
Parts:
- renumbered D9 to D10, J1 to J2, P23 to P22, R23 to R24, R24 to R25
Changed lines of the file:
@@
 LIBS:zetex
 LIBS:Zilog
-LIBS:KERISE-cache
 EELAYER 25 0
 EELAYER END
 $Descr A4 11693 8268
 encoding utf-8
-Sheet 11 13
+Sheet 11 15
 Title ""
 Date ""
@@
 BAT_OUT
 $Comp
-L R_Small R23
+L R_Small R24
 U 1 1 592C8650
 P 5000 5200
-F 0 "R23" H 5030 5220 50  0000 L CNN
+F 0 "R24" H 5030 5220 50  0000 L CNN
 F 1 "4.7k" H 5030 5160 50  0000 L CNN
 F 2 "Resistors_SMD:R_0402" H 5000 5200 50  0001 C CNN
@@
 $EndComp
 $Comp
-L R_Small R24
+L R_Small R25
 U 1 1 592C9443
 P 6300 5000
-F 0 "R24" H 6330 5020 50  0000 L CNN
+F 0 "R25" H 6330 5020 50  0000 L CNN
 F 1 "10k" H 6330 4960 50  0000 L CNN
 F 2 "Resistors_SMD:R_0402" H 6300 5000 50  0001 C CNN
@@
 $EndComp
 $Comp
-L LED_Small D9
+L LED_Small D10
 U 1 1 592C9513
 P 6600 5000
-F 0 "D9" H 6550 5125 50  0000 L CNN
+F 0 "D10" H 6550 5125 50  0000 L CNN
 F 1 "Status" H 6500 4900 50  0000 L CNN
 F 2 "LEDs:LED_0402" V 6600 5000 50  0001 C CNN
@@
 $EndComp
 $Comp
-L USB_OTG J1
+L USB_OTG J2
 U 1 1 5942A7E5
 P 4700 2300
-F 0 "J1" H 4500 2750 50  0000 L CNN
+F 0 "J2" H 4500 2750 50  0000 L CNN
 F 1 "USB_OTG" H 4500 2650 50  0000 L CNN
 F 2 "mouse:ZX62R-B-5P" H 4850 2250 50  0001 C CNN
@@
 NoConn ~ 5000 2500
 $Comp
-L CONN_01X04 P23
+L CONN_01X04 P22
 U 1 1 592C5604
 P 7000 2450
-F 0 "P23" H 7000 2700 50  0000 C CNN
+F 0 "P22" H 7000 2700 50  0000 C CNN
 F 1 "COM" V 7100 2450 50  0000 C CNN
 F 2 "Socket_Strips:Socket_Strip_Straight_1x04_Pitch1.27mm" H 7000 2450 50  0001 C CNN
