File: kicad/Encoder.sch (KiCad schematic (older format))
At the start: 4 parts, among them P19 ENC_Host, P20 ENC_Slave, U8 AS5048A

Commit message: 4輪の改良版を設計
Parts:
- renumbered P19 to P18, P20 to P19
Changed lines of the file:
@@
 LIBS:zetex
 LIBS:Zilog
-LIBS:KERISE-cache
 EELAYER 25 0
 EELAYER END
 $Descr A4 11693 8268
 encoding utf-8
-Sheet 9 13
+Sheet 9 14
 Title ""
 Date ""
@@
 P 4100 3600
 AR Path="/592ADBF2/589E94E9" Ref="#PWR057"  Part="1"
-AR Path="/59347BCD/589E94E9" Ref="#PWR068"  Part="1"
-F 0 "#PWR068" H 4100 3350 50  0001 C CNN
+AR Path="/59347BCD/589E94E9" Ref="#PWR065"  Part="1"
+F 0 "#PWR065" H 4100 3350 50  0001 C CNN
 F 1 "GND" H 4100 3450 50  0000 C CNN
 F 2 "" H 4100 3600 50  0000 C CNN
@@
 P 5100 2900
 AR Path="/592ADBF2/58CB39A3" Ref="#FLG058"  Part="1"
-AR Path="/59347BCD/58CB39A3" Ref="#FLG069"  Part="1"
-F 0 "#FLG069" H 5100 2995 50  0001 C CNN
+AR Path="/59347BCD/58CB39A3" Ref="#FLG066"  Part="1"
+F 0 "#FLG066" H 5100 2995 50  0001 C CNN
 F 1 "PWR_FLAG" H 5100 3080 50  0000 C CNN
 F 2 "" H 5100 2900 50  0000 C CNN
@@
 P 5100 3600
 AR Path="/592ADBF2/58CB39EE" Ref="#FLG059"  Part="1"
-AR Path="/59347BCD/58CB39EE" Ref="#FLG070"  Part="1"
-F 0 "#FLG070" H 5100 3695 50  0001 C CNN
+AR Path="/59347BCD/58CB39EE" Ref="#FLG067"  Part="1"
+F 0 "#FLG067" H 5100 3695 50  0001 C CNN
 F 1 "PWR_FLAG" H 5100 3780 50  0000 C CNN
 F 2 "" H 5100 3600 50  0000 C CNN
@@
 P 4100 2900
 AR Path="/592ADBF2/589CCACF" Ref="#PWR060"  Part="1"
-AR Path="/59347BCD/589CCACF" Ref="#PWR071"  Part="1"
-F 0 "#PWR071" H 4100 2750 50  0001 C CNN
+AR Path="/59347BCD/589CCACF" Ref="#PWR068"  Part="1"
+F 0 "#PWR068" H 4100 2750 50  0001 C CNN
 F 1 "+3.3V" H 4100 3040 50  0000 C CNN
 F 2 "" H 4100 2900 50  0000 C CNN
@@
 P 5700 2900
 AR Path="/592ADBF2/592A96DD" Ref="C26"  Part="1"
-AR Path="/59347BCD/592A96DD" Ref="C33"  Part="1"
-F 0 "C33" H 5710 2970 50  0000 L CNN
+AR Path="/59347BCD/592A96DD" Ref="C29"  Part="1"
+F 0 "C29" H 5710 2970 50  0000 L CNN
 F 1 "0.1u" H 5710 2820 50  0000 L CNN
 F 2 "Capacitors_SMD:C_0201" H 5700 2900 50  0001 C CNN
@@
 P 6400 2900
 AR Path="/592ADBF2/5933FF2E" Ref="U8"  Part="1"
-AR Path="/59347BCD/5933FF2E" Ref="U12"  Part="1"
-F 0 "U12" H 6400 3450 60  0000 C CNN
+AR Path="/59347BCD/5933FF2E" Ref="U10"  Part="1"
+F 0 "U10" H 6400 3450 60  0000 C CNN
 F 1 "AS5048A" H 6400 3300 60  0000 C CNN
 F 2 "mouse:TSSOP-14_4.4x5mm_Pitch0.65mm" H 6400 3300 60  0001 C CNN
@@
 $EndComp
 $Comp
-L CONN_01X06 P20
+L CONN_01X06 P19
 U 1 1 59340164
 P 4800 3250
-AR Path="/592ADBF2/59340164" Ref="P20"  Part="1"
-AR Path="/59347BCD/59340164" Ref="P25"  Part="1"
-F 0 "P25" H 4800 3600 50  0000 C CNN
+AR Path="/592ADBF2/59340164" Ref="P19"  Part="1"
+AR Path="/59347BCD/59340164" Ref="P23"  Part="1"
+F 0 "P23" H 4800 3600 50  0000 C CNN
 F 1 "ENC_Slave" V 4900 3250 50  0000 C CNN
 F 2 "mouse:STAND_AS_SLAVE" H 4800 3250 50  0001 C CNN
@@
 	5000 3100 5100 3100
 $Comp
-L CONN_01X06 P19
+L CONN_01X06 P18
 U 1 1 59340673
 P 4400 3250
-AR Path="/592ADBF2/59340673" Ref="P19"  Part="1"
-AR Path="/59347BCD/59340673" Ref="P24"  Part="1"
-F 0 "P24" H 4400 3600 50  0000 C CNN
+AR Path="/592ADBF2/59340673" Ref="P18"  Part="1"
+AR Path="/59347BCD/59340673" Ref="P22"  Part="1"
+F 0 "P22" H 4400 3600 50  0000 C CNN
 F 1 "ENC_Host" V 4500 3250 50  0000 C CNN
 F 2 "mouse:STAND_AS_HOST" H 4400 3250 50  0001 C CNN

Commit message: 部品を配置
Connections:
- net CS: now also P18.5 (P5); no longer P18.2 (P2)
- net MISO: now also P18.3 (P3); no longer P18.4 (P4)
- net MOSI: now also P18.2 (P2); no longer P18.5 (P5)
- net SCLK: now also P18.4 (P4); no longer P18.3 (P3)
- net s_CS: now also P19.5 (P5); no longer P19.2 (P2)
- net s_MISO: now also P19.3 (P3); no longer P19.4 (P4)
- net s_MOSI: now also P19.2 (P2); no longer P19.5 (P5)
- net s_SCLK: now also P19.4 (P4); no longer P19.3 (P3)
Changed lines of the file:
@@
 AR Path="/592ADBF2/589E94E9" Ref="#PWR057"  Part="1"
 AR Path="/59347BCD/589E94E9" Ref="#PWR065"  Part="1"
-F 0 "#PWR065" H 4100 3350 50  0001 C CNN
+F 0 "#PWR057" H 4100 3350 50  0001 C CNN
 F 1 "GND" H 4100 3450 50  0000 C CNN
 F 2 "" H 4100 3600 50  0000 C CNN
@@
 	1    0    0    -1
 $EndComp
-Text HLabel 4100 3100 0    60   Input ~ 0
+Text HLabel 4100 3400 0    60   Input ~ 0
 CS
 $Comp
@@
 AR Path="/592ADBF2/58CB39A3" Ref="#FLG058"  Part="1"
 AR Path="/59347BCD/58CB39A3" Ref="#FLG066"  Part="1"
-F 0 "#FLG066" H 5100 2995 50  0001 C CNN
+F 0 "#FLG058" H 5100 2995 50  0001 C CNN
 F 1 "PWR_FLAG" H 5100 3080 50  0000 C CNN
 F 2 "" H 5100 2900 50  0000 C CNN
@@
 AR Path="/592ADBF2/58CB39EE" Ref="#FLG059"  Part="1"
 AR Path="/59347BCD/58CB39EE" Ref="#FLG067"  Part="1"
-F 0 "#FLG067" H 5100 3695 50  0001 C CNN
+F 0 "#FLG059" H 5100 3695 50  0001 C CNN
 F 1 "PWR_FLAG" H 5100 3780 50  0000 C CNN
 F 2 "" H 5100 3600 50  0000 C CNN
@@
 AR Path="/592ADBF2/589CCACF" Ref="#PWR060"  Part="1"
 AR Path="/59347BCD/589CCACF" Ref="#PWR068"  Part="1"
-F 0 "#PWR068" H 4100 2750 50  0001 C CNN
+F 0 "#PWR060" H 4100 2750 50  0001 C CNN
 F 1 "+3.3V" H 4100 3040 50  0000 C CNN
 F 2 "" H 4100 2900 50  0000 C CNN
@@
 AR Path="/592ADBF2/592A96DD" Ref="C26"  Part="1"
 AR Path="/59347BCD/592A96DD" Ref="C29"  Part="1"
-F 0 "C29" H 5710 2970 50  0000 L CNN
+F 0 "C26" H 5710 2970 50  0000 L CNN
 F 1 "0.1u" H 5710 2820 50  0000 L CNN
 F 2 "Capacitors_SMD:C_0201" H 5700 2900 50  0001 C CNN
@@
 AR Path="/592ADBF2/5933FF2E" Ref="U8"  Part="1"
 AR Path="/59347BCD/5933FF2E" Ref="U10"  Part="1"
-F 0 "U10" H 6400 3450 60  0000 C CNN
+F 0 "U8" H 6400 3450 60  0000 C CNN
 F 1 "AS5048A" H 6400 3300 60  0000 C CNN
 F 2 "mouse:TSSOP-14_4.4x5mm_Pitch0.65mm" H 6400 3300 60  0001 C CNN
@@
 AR Path="/592ADBF2/59340164" Ref="P19"  Part="1"
 AR Path="/59347BCD/59340164" Ref="P23"  Part="1"
-F 0 "P23" H 4800 3600 50  0000 C CNN
+F 0 "P19" H 4800 3600 50  0000 C CNN
 F 1 "ENC_Slave" V 4900 3250 50  0000 C CNN
 F 2 "mouse:STAND_AS_SLAVE" H 4800 3250 50  0001 C CNN
@@
 Text Label 6900 2900 0    60   ~ 0
 s_MOSI
+Text Label 5100 3400 0    60   ~ 0
+s_CS
+Text Label 5100 3300 0    60   ~ 0
+s_SCLK
+Text Label 5100 3200 0    60   ~ 0
+s_MISO
 Text Label 5100 3100 0    60   ~ 0
-s_CS
-Text Label 5100 3200 0    60   ~ 0
-s_SCLK
-Text Label 5100 3300 0    60   ~ 0
-s_MISO
-Text Label 5100 3400 0    60   ~ 0
 s_MOSI
 Wire Wire Line
@@
 AR Path="/592ADBF2/59340673" Ref="P18"  Part="1"
 AR Path="/59347BCD/59340673" Ref="P22"  Part="1"
-F 0 "P22" H 4400 3600 50  0000 C CNN
+F 0 "P18" H 4400 3600 50  0000 C CNN
 F 1 "ENC_Host" V 4500 3250 50  0000 C CNN
 F 2 "mouse:STAND_AS_HOST" H 4400 3250 50  0001 C CNN
@@
 	1    0    0    -1
 $EndComp
+Text HLabel 4100 3300 0    60   Input ~ 0
+SCLK
 Text HLabel 4100 3200 0    60   Input ~ 0
-SCLK
-Text HLabel 4100 3300 0    60   Input ~ 0
 MISO
-Text HLabel 4100 3400 0    60   Input ~ 0
+Text HLabel 4100 3100 0    60   Input ~ 0
 MOSI
 Wire Wire Line

Commit message: 細部を改良，自動配線成功
Connections:
- net CS: now also P18.2 (P2); no longer P18.5 (P5)
- net MISO: now also P18.5 (P5); no longer P18.3 (P3)
- net MOSI: now also P18.4 (P4); no longer P18.2 (P2)
- net SCLK: now also P18.3 (P3); no longer P18.4 (P4)
- net s_CS: now also P19.2 (P2); no longer P19.5 (P5)
- net s_MISO: now also P19.5 (P5); no longer P19.3 (P3)
- net s_MOSI: now also P19.4 (P4); no longer P19.2 (P2)
- net s_SCLK: now also P19.3 (P3); no longer P19.4 (P4)
Changed lines of the file:
@@
 LIBS:zetex
 LIBS:Zilog
+LIBS:KERISE-cache
 EELAYER 25 0
 EELAYER END
 $Descr A4 11693 8268
 encoding utf-8
-Sheet 9 14
+Sheet 11 14
 Title ""
 Date ""
@@
 AR Path="/592ADBF2/589E94E9" Ref="#PWR057"  Part="1"
 AR Path="/59347BCD/589E94E9" Ref="#PWR065"  Part="1"
-F 0 "#PWR057" H 4100 3350 50  0001 C CNN
+F 0 "#PWR065" H 4100 3350 50  0001 C CNN
 F 1 "GND" H 4100 3450 50  0000 C CNN
 F 2 "" H 4100 3600 50  0000 C CNN
@@
 	1    0    0    -1
 $EndComp
-Text HLabel 4100 3400 0    60   Input ~ 0
+Text HLabel 4100 3100 0    60   Input ~ 0
 CS
 $Comp
@@
 AR Path="/592ADBF2/58CB39A3" Ref="#FLG058"  Part="1"
 AR Path="/59347BCD/58CB39A3" Ref="#FLG066"  Part="1"
-F 0 "#FLG058" H 5100 2995 50  0001 C CNN
+F 0 "#FLG066" H 5100 2995 50  0001 C CNN
 F 1 "PWR_FLAG" H 5100 3080 50  0000 C CNN
 F 2 "" H 5100 2900 50  0000 C CNN
@@
 AR Path="/592ADBF2/58CB39EE" Ref="#FLG059"  Part="1"
 AR Path="/59347BCD/58CB39EE" Ref="#FLG067"  Part="1"
-F 0 "#FLG059" H 5100 3695 50  0001 C CNN
+F 0 "#FLG067" H 5100 3695 50  0001 C CNN
 F 1 "PWR_FLAG" H 5100 3780 50  0000 C CNN
 F 2 "" H 5100 3600 50  0000 C CNN
@@
 AR Path="/592ADBF2/589CCACF" Ref="#PWR060"  Part="1"
 AR Path="/59347BCD/589CCACF" Ref="#PWR068"  Part="1"
-F 0 "#PWR060" H 4100 2750 50  0001 C CNN
+F 0 "#PWR068" H 4100 2750 50  0001 C CNN
 F 1 "+3.3V" H 4100 3040 50  0000 C CNN
 F 2 "" H 4100 2900 50  0000 C CNN
@@
 AR Path="/592ADBF2/592A96DD" Ref="C26"  Part="1"
 AR Path="/59347BCD/592A96DD" Ref="C29"  Part="1"
-F 0 "C26" H 5710 2970 50  0000 L CNN
+F 0 "C29" H 5710 2970 50  0000 L CNN
 F 1 "0.1u" H 5710 2820 50  0000 L CNN
 F 2 "Capacitors_SMD:C_0201" H 5700 2900 50  0001 C CNN
@@
 AR Path="/592ADBF2/5933FF2E" Ref="U8"  Part="1"
 AR Path="/59347BCD/5933FF2E" Ref="U10"  Part="1"
-F 0 "U8" H 6400 3450 60  0000 C CNN
+F 0 "U10" H 6400 3450 60  0000 C CNN
 F 1 "AS5048A" H 6400 3300 60  0000 C CNN
 F 2 "mouse:TSSOP-14_4.4x5mm_Pitch0.65mm" H 6400 3300 60  0001 C CNN
@@
 AR Path="/592ADBF2/59340164" Ref="P19"  Part="1"
 AR Path="/59347BCD/59340164" Ref="P23"  Part="1"
-F 0 "P19" H 4800 3600 50  0000 C CNN
+F 0 "P23" H 4800 3600 50  0000 C CNN
 F 1 "ENC_Slave" V 4900 3250 50  0000 C CNN
 F 2 "mouse:STAND_AS_SLAVE" H 4800 3250 50  0001 C CNN
@@
 Text Label 6900 2900 0    60   ~ 0
 s_MOSI
+Text Label 5100 3100 0    60   ~ 0
+s_CS
+Text Label 5100 3200 0    60   ~ 0
+s_SCLK
 Text Label 5100 3400 0    60   ~ 0
-s_CS
+s_MISO
 Text Label 5100 3300 0    60   ~ 0
-s_SCLK
-Text Label 5100 3200 0    60   ~ 0
-s_MISO
-Text Label 5100 3100 0    60   ~ 0
 s_MOSI
 Wire Wire Line
@@
 AR Path="/592ADBF2/59340673" Ref="P18"  Part="1"
 AR Path="/59347BCD/59340673" Ref="P22"  Part="1"
-F 0 "P18" H 4400 3600 50  0000 C CNN
+F 0 "P22" H 4400 3600 50  0000 C CNN
 F 1 "ENC_Host" V 4500 3250 50  0000 C CNN
 F 2 "mouse:STAND_AS_HOST" H 4400 3250 50  0001 C CNN
@@
 	1    0    0    -1
 $EndComp
+Text HLabel 4100 3200 0    60   Input ~ 0
+SCLK
+Text HLabel 4100 3400 0    60   Input ~ 0
+MISO
 Text HLabel 4100 3300 0    60   Input ~ 0
-SCLK
-Text HLabel 4100 3200 0    60   Input ~ 0
-MISO
-Text HLabel 4100 3100 0    60   Input ~ 0
 MOSI
 Wire Wire Line

Commit message: 回路とフットプリントを改良
Parts:
- renumbered C26 to C28
Changed lines of the file:
@@
 $EndDescr
 $Comp
-L GND #PWR057
+L GND #PWR062
 U 1 1 589E94E9
 P 4100 3600
-AR Path="/592ADBF2/589E94E9" Ref="#PWR057"  Part="1"
-AR Path="/59347BCD/589E94E9" Ref="#PWR065"  Part="1"
-F 0 "#PWR065" H 4100 3350 50  0001 C CNN
+AR Path="/592ADBF2/589E94E9" Ref="#PWR062"  Part="1"
+AR Path="/59347BCD/589E94E9" Ref="#PWR070"  Part="1"
+F 0 "#PWR070" H 4100 3350 50  0001 C CNN
 F 1 "GND" H 4100 3450 50  0000 C CNN
 F 2 "" H 4100 3600 50  0000 C CNN
@@
 CS
 $Comp
-L PWR_FLAG #FLG058
+L PWR_FLAG #FLG063
 U 1 1 58CB39A3
 P 5100 2900
-AR Path="/592ADBF2/58CB39A3" Ref="#FLG058"  Part="1"
-AR Path="/59347BCD/58CB39A3" Ref="#FLG066"  Part="1"
-F 0 "#FLG066" H 5100 2995 50  0001 C CNN
+AR Path="/592ADBF2/58CB39A3" Ref="#FLG063"  Part="1"
+AR Path="/59347BCD/58CB39A3" Ref="#FLG071"  Part="1"
+F 0 "#FLG071" H 5100 2995 50  0001 C CNN
 F 1 "PWR_FLAG" H 5100 3080 50  0000 C CNN
 F 2 "" H 5100 2900 50  0000 C CNN
@@
 $EndComp
 $Comp
-L PWR_FLAG #FLG059
+L PWR_FLAG #FLG064
 U 1 1 58CB39EE
 P 5100 3600
-AR Path="/592ADBF2/58CB39EE" Ref="#FLG059"  Part="1"
-AR Path="/59347BCD/58CB39EE" Ref="#FLG067"  Part="1"
-F 0 "#FLG067" H 5100 3695 50  0001 C CNN
+AR Path="/592ADBF2/58CB39EE" Ref="#FLG064"  Part="1"
+AR Path="/59347BCD/58CB39EE" Ref="#FLG072"  Part="1"
+F 0 "#FLG072" H 5100 3695 50  0001 C CNN
 F 1 "PWR_FLAG" H 5100 3780 50  0000 C CNN
 F 2 "" H 5100 3600 50  0000 C CNN
@@
 $EndComp
 $Comp
-L +3.3V #PWR060
+L +3.3V #PWR065
 U 1 1 589CCACF
 P 4100 2900
-AR Path="/592ADBF2/589CCACF" Ref="#PWR060"  Part="1"
-AR Path="/59347BCD/589CCACF" Ref="#PWR068"  Part="1"
-F 0 "#PWR068" H 4100 2750 50  0001 C CNN
+AR Path="/592ADBF2/589CCACF" Ref="#PWR065"  Part="1"
+AR Path="/59347BCD/589CCACF" Ref="#PWR073"  Part="1"
+F 0 "#PWR073" H 4100 2750 50  0001 C CNN
 F 1 "+3.3V" H 4100 3040 50  0000 C CNN
 F 2 "" H 4100 2900 50  0000 C CNN
@@
 	4100 3500 4200 3500
 $Comp
-L C_Small C26
+L C_Small C28
 U 1 1 592A96DD
 P 5700 2900
-AR Path="/592ADBF2/592A96DD" Ref="C26"  Part="1"
-AR Path="/59347BCD/592A96DD" Ref="C29"  Part="1"
-F 0 "C29" H 5710 2970 50  0000 L CNN
+AR Path="/592ADBF2/592A96DD" Ref="C28"  Part="1"
+AR Path="/59347BCD/592A96DD" Ref="C31"  Part="1"
+F 0 "C31" H 5710 2970 50  0000 L CNN
 F 1 "0.1u" H 5710 2820 50  0000 L CNN
 F 2 "Capacitors_SMD:C_0201" H 5700 2900 50  0001 C CNN

Commit message: 自動配線1残し
Parts:
- renumbered C28 to C27, P18 to P10, P19 to P11
Changed lines of the file:
@@
 $EndDescr
 $Comp
-L GND #PWR062
+L GND #PWR063
 U 1 1 589E94E9
 P 4100 3600
-AR Path="/592ADBF2/589E94E9" Ref="#PWR062"  Part="1"
-AR Path="/59347BCD/589E94E9" Ref="#PWR070"  Part="1"
-F 0 "#PWR070" H 4100 3350 50  0001 C CNN
+AR Path="/592ADBF2/589E94E9" Ref="#PWR063"  Part="1"
+AR Path="/59347BCD/589E94E9" Ref="#PWR071"  Part="1"
+F 0 "#PWR071" H 4100 3350 50  0001 C CNN
 F 1 "GND" H 4100 3450 50  0000 C CNN
 F 2 "" H 4100 3600 50  0000 C CNN
@@
 CS
 $Comp
-L PWR_FLAG #FLG063
+L PWR_FLAG #FLG064
 U 1 1 58CB39A3
 P 5100 2900
-AR Path="/592ADBF2/58CB39A3" Ref="#FLG063"  Part="1"
-AR Path="/59347BCD/58CB39A3" Ref="#FLG071"  Part="1"
-F 0 "#FLG071" H 5100 2995 50  0001 C CNN
+AR Path="/592ADBF2/58CB39A3" Ref="#FLG064"  Part="1"
+AR Path="/59347BCD/58CB39A3" Ref="#FLG072"  Part="1"
+F 0 "#FLG072" H 5100 2995 50  0001 C CNN
 F 1 "PWR_FLAG" H 5100 3080 50  0000 C CNN
 F 2 "" H 5100 2900 50  0000 C CNN
@@
 $EndComp
 $Comp
-L PWR_FLAG #FLG064
+L PWR_FLAG #FLG065
 U 1 1 58CB39EE
 P 5100 3600
-AR Path="/592ADBF2/58CB39EE" Ref="#FLG064"  Part="1"
-AR Path="/59347BCD/58CB39EE" Ref="#FLG072"  Part="1"
-F 0 "#FLG072" H 5100 3695 50  0001 C CNN
+AR Path="/592ADBF2/58CB39EE" Ref="#FLG065"  Part="1"
+AR Path="/59347BCD/58CB39EE" Ref="#FLG073"  Part="1"
+F 0 "#FLG073" H 5100 3695 50  0001 C CNN
 F 1 "PWR_FLAG" H 5100 3780 50  0000 C CNN
 F 2 "" H 5100 3600 50  0000 C CNN
@@
 $EndComp
 $Comp
-L +3.3V #PWR065
+L +3.3V #PWR066
 U 1 1 589CCACF
 P 4100 2900
-AR Path="/592ADBF2/589CCACF" Ref="#PWR065"  Part="1"
-AR Path="/59347BCD/589CCACF" Ref="#PWR073"  Part="1"
-F 0 "#PWR073" H 4100 2750 50  0001 C CNN
+AR Path="/592ADBF2/589CCACF" Ref="#PWR066"  Part="1"
+AR Path="/59347BCD/589CCACF" Ref="#PWR074"  Part="1"
+F 0 "#PWR074" H 4100 2750 50  0001 C CNN
 F 1 "+3.3V" H 4100 3040 50  0000 C CNN
 F 2 "" H 4100 2900 50  0000 C CNN
@@
 	4100 3500 4200 3500
 $Comp
-L C_Small C28
+L C_Small C27
 U 1 1 592A96DD
 P 5700 2900
-AR Path="/592ADBF2/592A96DD" Ref="C28"  Part="1"
-AR Path="/59347BCD/592A96DD" Ref="C31"  Part="1"
-F 0 "C31" H 5710 2970 50  0000 L CNN
+AR Path="/592ADBF2/592A96DD" Ref="C27"  Part="1"
+AR Path="/59347BCD/592A96DD" Ref="C30"  Part="1"
+F 0 "C30" H 5710 2970 50  0000 L CNN
 F 1 "0.1u" H 5710 2820 50  0000 L CNN
 F 2 "Capacitors_SMD:C_0201" H 5700 2900 50  0001 C CNN
@@
 $EndComp
 $Comp
-L CONN_01X06 P19
+L CONN_01X06 P11
 U 1 1 59340164
 P 4800 3250
-AR Path="/592ADBF2/59340164" Ref="P19"  Part="1"
-AR Path="/59347BCD/59340164" Ref="P23"  Part="1"
-F 0 "P23" H 4800 3600 50  0000 C CNN
+AR Path="/592ADBF2/59340164" Ref="P11"  Part="1"
+AR Path="/59347BCD/59340164" Ref="P15"  Part="1"
+F 0 "P15" H 4800 3600 50  0000 C CNN
 F 1 "ENC_Slave" V 4900 3250 50  0000 C CNN
 F 2 "mouse:STAND_AS_SLAVE" H 4800 3250 50  0001 C CNN
@@
 	5000 3100 5100 3100
 $Comp
-L CONN_01X06 P18
+L CONN_01X06 P10
 U 1 1 59340673
 P 4400 3250
-AR Path="/592ADBF2/59340673" Ref="P18"  Part="1"
-AR Path="/59347BCD/59340673" Ref="P22"  Part="1"
-F 0 "P22" H 4400 3600 50  0000 C CNN
+AR Path="/592ADBF2/59340673" Ref="P10"  Part="1"
+AR Path="/59347BCD/59340673" Ref="P14"  Part="1"
+F 0 "P14" H 4400 3600 50  0000 C CNN
 F 1 "ENC_Host" V 4500 3250 50  0000 C CNN
 F 2 "mouse:STAND_AS_HOST" H 4400 3250 50  0001 C CNN

Commit message: 実装経験をもとにフットプリントを改良，ミスを修正
SC70サイズのオペアンプのピンアサインを修正
Parts:
- renumbered P11 to P10, P10 to P9
Changed lines of the file:
@@
 $Descr A4 11693 8268
 encoding utf-8
-Sheet 11 14
+Sheet 9 14
 Title ""
 Date ""
@@
 $EndDescr
 $Comp
-L GND #PWR063
+L GND #PWR58
 U 1 1 589E94E9
 P 4100 3600
-AR Path="/592ADBF2/589E94E9" Ref="#PWR063"  Part="1"
-AR Path="/59347BCD/589E94E9" Ref="#PWR071"  Part="1"
-F 0 "#PWR071" H 4100 3350 50  0001 C CNN
+AR Path="/592ADBF2/589E94E9" Ref="#PWR58"  Part="1"
+AR Path="/59347BCD/589E94E9" Ref="#PWR62"  Part="1"
+F 0 "#PWR62" H 4100 3350 50  0001 C CNN
 F 1 "GND" H 4100 3450 50  0000 C CNN
 F 2 "" H 4100 3600 50  0000 C CNN
@@
 CS
 $Comp
-L PWR_FLAG #FLG064
+L PWR_FLAG #FLG7
 U 1 1 58CB39A3
 P 5100 2900
-AR Path="/592ADBF2/58CB39A3" Ref="#FLG064"  Part="1"
-AR Path="/59347BCD/58CB39A3" Ref="#FLG072"  Part="1"
-F 0 "#FLG072" H 5100 2995 50  0001 C CNN
+AR Path="/592ADBF2/58CB39A3" Ref="#FLG7"  Part="1"
+AR Path="/59347BCD/58CB39A3" Ref="#FLG11"  Part="1"
+F 0 "#FLG11" H 5100 2995 50  0001 C CNN
 F 1 "PWR_FLAG" H 5100 3080 50  0000 C CNN
 F 2 "" H 5100 2900 50  0000 C CNN
@@
 $EndComp
 $Comp
-L PWR_FLAG #FLG065
+L PWR_FLAG #FLG8
 U 1 1 58CB39EE
 P 5100 3600
-AR Path="/592ADBF2/58CB39EE" Ref="#FLG065"  Part="1"
-AR Path="/59347BCD/58CB39EE" Ref="#FLG073"  Part="1"
-F 0 "#FLG073" H 5100 3695 50  0001 C CNN
+AR Path="/592ADBF2/58CB39EE" Ref="#FLG8"  Part="1"
+AR Path="/59347BCD/58CB39EE" Ref="#FLG12"  Part="1"
+F 0 "#FLG12" H 5100 3695 50  0001 C CNN
 F 1 "PWR_FLAG" H 5100 3780 50  0000 C CNN
 F 2 "" H 5100 3600 50  0000 C CNN
@@
 $EndComp
 $Comp
-L +3.3V #PWR066
+L +3.3V #PWR57
 U 1 1 589CCACF
 P 4100 2900
-AR Path="/592ADBF2/589CCACF" Ref="#PWR066"  Part="1"
-AR Path="/59347BCD/589CCACF" Ref="#PWR074"  Part="1"
-F 0 "#PWR074" H 4100 2750 50  0001 C CNN
+AR Path="/592ADBF2/589CCACF" Ref="#PWR57"  Part="1"
+AR Path="/59347BCD/589CCACF" Ref="#PWR61"  Part="1"
+F 0 "#PWR61" H 4100 2750 50  0001 C CNN
 F 1 "+3.3V" H 4100 3040 50  0000 C CNN
 F 2 "" H 4100 2900 50  0000 C CNN
@@
 $EndComp
 $Comp
-L CONN_01X06 P11
+L CONN_01X06 P10
 U 1 1 59340164
 P 4800 3250
-AR Path="/592ADBF2/59340164" Ref="P11"  Part="1"
-AR Path="/59347BCD/59340164" Ref="P15"  Part="1"
-F 0 "P15" H 4800 3600 50  0000 C CNN
+AR Path="/592ADBF2/59340164" Ref="P10"  Part="1"
+AR Path="/59347BCD/59340164" Ref="P14"  Part="1"
+F 0 "P14" H 4800 3600 50  0000 C CNN
 F 1 "ENC_Slave" V 4900 3250 50  0000 C CNN
 F 2 "mouse:STAND_AS_SLAVE" H 4800 3250 50  0001 C CNN
@@
 	5000 3100 5100 3100
 $Comp
-L CONN_01X06 P10
+L CONN_01X06 P9
 U 1 1 59340673
 P 4400 3250
-AR Path="/592ADBF2/59340673" Ref="P10"  Part="1"
-AR Path="/59347BCD/59340673" Ref="P14"  Part="1"
-F 0 "P14" H 4400 3600 50  0000 C CNN
+AR Path="/592ADBF2/59340673" Ref="P9"  Part="1"
+AR Path="/59347BCD/59340673" Ref="P13"  Part="1"
+F 0 "P13" H 4400 3600 50  0000 C CNN
 F 1 "ENC_Host" V 4500 3250 50  0000 C CNN
 F 2 "mouse:STAND_AS_HOST" H 4400 3250 50  0001 C CNN
