File: kicad/Fan.sch (KiCad schematic (older format))
At the start: 3 parts, among them P18 Fan, Q4 IRFML8244

Commit message: 4輪の改良版を設計
Parts:
- Q4: value IRFML8244 -> DMN3065LW-7; footprint TO_SOT_Packages_SMD:SOT-23 -> TO_SOT_Packages_SMD:SOT-323_SC-70
- renumbered P18 to P17, R20 to R21
Changed lines of the file:
@@
 LIBS:zetex
 LIBS:Zilog
-LIBS:KERISE-cache
 EELAYER 25 0
 EELAYER END
 $Descr A4 11693 8268
 encoding utf-8
-Sheet 8 13
+Sheet 8 14
 Title ""
 Date ""
@@
 P 5050 4800
 F 0 "Q4" H 5350 4850 50  0000 R CNN
-F 1 "IRFML8244" H 5700 4750 50  0000 R CNN
-F 2 "TO_SOT_Packages_SMD:SOT-23" H 5250 4900 50  0001 C CNN
+F 1 "DMN3065LW-7" H 5800 4750 50  0000 R CNN
+F 2 "TO_SOT_Packages_SMD:SOT-323_SC-70" H 5250 4900 50  0001 C CNN
 F 3 "" H 5050 4800 50  0000 C CNN
 	1    5050 4800
@@
 	5150 5000 5150 5300
 $Comp
-L R R20
+L R R21
 U 1 1 58AB90F7
 P 4750 5050
-F 0 "R20" V 4830 5050 50  0000 C CNN
+F 0 "R21" V 4830 5050 50  0000 C CNN
 F 1 "10k" V 4750 5050 50  0000 C CNN
 F 2 "Resistors_SMD:R_0201" V 4680 5050 50  0001 C CNN
@@
 	4750 5300 4750 5200
 $Comp
-L CONN_01X02 P18
+L CONN_01X02 P17
 U 1 1 58AB920C
 P 5450 4350
-F 0 "P18" H 5450 4500 50  0000 C CNN
+F 0 "P17" H 5450 4500 50  0000 C CNN
 F 1 "Fan" V 5550 4350 50  0000 C CNN
 F 2 "mouse:SMD_conn_2" H 5450 4350 50  0001 C CNN

Commit message: 自動配線1残し
Parts:
- renumbered P17 to P9, R21 to R22
Changed lines of the file:
@@
 $EndComp
 $Comp
-L GND #PWR059
+L GND #PWR060
 U 1 1 58AB90DB
 P 5150 5300
-F 0 "#PWR059" H 5150 5050 50  0001 C CNN
+F 0 "#PWR060" H 5150 5050 50  0001 C CNN
 F 1 "GND" H 5150 5150 50  0000 C CNN
 F 2 "" H 5150 5300 50  0000 C CNN
@@
 	5150 5000 5150 5300
 $Comp
-L R R21
+L R R22
 U 1 1 58AB90F7
 P 4750 5050
-F 0 "R21" V 4830 5050 50  0000 C CNN
+F 0 "R22" V 4830 5050 50  0000 C CNN
 F 1 "10k" V 4750 5050 50  0000 C CNN
 F 2 "Resistors_SMD:R_0201" V 4680 5050 50  0001 C CNN
@@
 Connection ~ 4750 4800
 $Comp
-L GND #PWR060
+L GND #PWR061
 U 1 1 58AB9100
 P 4750 5300
-F 0 "#PWR060" H 4750 5050 50  0001 C CNN
+F 0 "#PWR061" H 4750 5050 50  0001 C CNN
 F 1 "GND" H 4750 5150 50  0000 C CNN
 F 2 "" H 4750 5300 50  0000 C CNN
@@
 	4750 5300 4750 5200
 $Comp
-L CONN_01X02 P17
+L CONN_01X02 P9
 U 1 1 58AB920C
 P 5450 4350
-F 0 "P17" H 5450 4500 50  0000 C CNN
+F 0 "P9" H 5450 4500 50  0000 C CNN
 F 1 "Fan" V 5550 4350 50  0000 C CNN
 F 2 "mouse:SMD_conn_2" H 5450 4350 50  0001 C CNN
@@
 $EndComp
 $Comp
-L +BATT #PWR061
+L +BATT #PWR062
 U 1 1 58AB927D
 P 5150 4100
-F 0 "#PWR061" H 5150 3950 50  0001 C CNN
+F 0 "#PWR062" H 5150 3950 50  0001 C CNN
 F 1 "+BATT" H 5150 4240 50  0000 C CNN
 F 2 "" H 5150 4100 50  0000 C CNN

Commit message: 実装経験をもとにフットプリントを改良，ミスを修正
SC70サイズのオペアンプのピンアサインを修正
Parts:
- renumbered P9 to P8
Changed lines of the file:
@@
 $EndComp
 $Comp
-L GND #PWR060
+L GND #PWR56
 U 1 1 58AB90DB
 P 5150 5300
-F 0 "#PWR060" H 5150 5050 50  0001 C CNN
+F 0 "#PWR56" H 5150 5050 50  0001 C CNN
 F 1 "GND" H 5150 5150 50  0000 C CNN
 F 2 "" H 5150 5300 50  0000 C CNN
@@
 Connection ~ 4750 4800
 $Comp
-L GND #PWR061
+L GND #PWR54
 U 1 1 58AB9100
 P 4750 5300
-F 0 "#PWR061" H 4750 5050 50  0001 C CNN
+F 0 "#PWR54" H 4750 5050 50  0001 C CNN
 F 1 "GND" H 4750 5150 50  0000 C CNN
 F 2 "" H 4750 5300 50  0000 C CNN
@@
 	4750 5300 4750 5200
 $Comp
-L CONN_01X02 P9
+L CONN_01X02 P8
 U 1 1 58AB920C
 P 5450 4350
-F 0 "P9" H 5450 4500 50  0000 C CNN
+F 0 "P8" H 5450 4500 50  0000 C CNN
 F 1 "Fan" V 5550 4350 50  0000 C CNN
 F 2 "mouse:SMD_conn_2" H 5450 4350 50  0001 C CNN
@@
 $EndComp
 $Comp
-L +BATT #PWR062
+L +BATT #PWR55
 U 1 1 58AB927D
 P 5150 4100
-F 0 "#PWR062" H 5150 3950 50  0001 C CNN
+F 0 "#PWR55" H 5150 3950 50  0001 C CNN
 F 1 "+BATT" H 5150 4240 50  0000 C CNN
 F 2 "" H 5150 4100 50  0000 C CNN
