File: kicad/ToF.sch (KiCad schematic (older format))
At the start: 7 parts, among them P21 ToF_Host, P22 ToF_Slave, U9 VL53L0X

Commit message: 4輪の改良版を設計
Parts:
- renumbered P21 to P20, P22 to P21, R21 to R22, R22 to R23
Changed lines of the file:
@@
 LIBS:zetex
 LIBS:Zilog
-LIBS:KERISE-cache
 EELAYER 25 0
 EELAYER END
 $Descr A4 11693 8268
 encoding utf-8
-Sheet 10 13
+Sheet 10 14
 Title ""
 Date ""
@@
 	5400 3300 5400 3400
 $Comp
-L CONN_01X04 P21
+L CONN_01X04 P20
 U 1 1 592AB778
 P 4600 2450
-F 0 "P21" H 4600 2700 50  0000 C CNN
+F 0 "P20" H 4600 2700 50  0000 C CNN
 F 1 "ToF_Host" V 4700 2450 50  0000 C CNN
 F 2 "mouse:STAND_PR_HOST" H 4600 2450 50  0001 C CNN
@@
 $EndComp
 $Comp
-L CONN_01X04 P22
+L CONN_01X04 P21
 U 1 1 592AB803
 P 5000 2450
-F 0 "P22" H 5000 2700 50  0000 C CNN
+F 0 "P21" H 5000 2700 50  0000 C CNN
 F 1 "ToF_Slave" V 5100 2450 50  0000 C CNN
 F 2 "mouse:STAND_PR_SLAVE" H 5000 2450 50  0001 C CNN
@@
 $EndComp
 $Comp
-L R_Small R21
+L R_Small R22
 U 1 1 5932174C
 P 5800 3500
-F 0 "R21" H 5830 3520 50  0000 L CNN
+F 0 "R22" H 5830 3520 50  0000 L CNN
 F 1 "4.7k" H 5830 3460 50  0000 L CNN
 F 2 "Resistors_SMD:R_0201" H 5800 3500 50  0001 C CNN
@@
 $EndComp
 $Comp
-L R_Small R22
+L R_Small R23
 U 1 1 593217CA
 P 6100 3500
-F 0 "R22" H 6130 3520 50  0000 L CNN
+F 0 "R23" H 6130 3520 50  0000 L CNN
 F 1 "4.7k" H 6130 3460 50  0000 L CNN
 F 2 "Resistors_SMD:R_0201" H 6100 3500 50  0001 C CNN

Commit message: 回路とフットプリントを改良
Parts:
- renumbered C27 to C29, C28 to C30
Changed lines of the file:
@@
 	5400 3400 5300 3400
 $Comp
-L C_Small C28
+L C_Small C30
 U 1 1 592BA26F
 P 3900 3800
-F 0 "C28" H 3910 3870 50  0000 L CNN
+F 0 "C30" H 3910 3870 50  0000 L CNN
 F 1 "0.1u" H 3910 3720 50  0000 L CNN
 F 2 "Capacitors_SMD:C_0201" H 3900 3800 50  0001 C CNN
@@
 $EndComp
 $Comp
-L C_Small C27
+L C_Small C29
 U 1 1 592BA2BF
 P 3600 3800
-F 0 "C27" H 3610 3870 50  0000 L CNN
+F 0 "C29" H 3610 3870 50  0000 L CNN
 F 1 "4.7u" H 3610 3720 50  0000 L CNN
 F 2 "Capacitors_SMD:C_0402" H 3600 3800 50  0001 C CNN
@@
 $EndComp
 $Comp
-L GND #PWR061
+L GND #PWR066
 U 1 1 592ABB63
 P 4300 2700
-F 0 "#PWR061" H 4300 2450 50  0001 C CNN
+F 0 "#PWR066" H 4300 2450 50  0001 C CNN
 F 1 "GND" H 4300 2550 50  0000 C CNN
 F 2 "" H 4300 2700 50  0000 C CNN
@@
 	4300 2600 4400 2600
 $Comp
-L +3.3V #PWR062
+L +3.3V #PWR067
 U 1 1 592ABB9F
 P 4300 2200
-F 0 "#PWR062" H 4300 2050 50  0001 C CNN
+F 0 "#PWR067" H 4300 2050 50  0001 C CNN
 F 1 "+3.3V" H 4300 2340 50  0000 C CNN
 F 2 "" H 4300 2200 50  0000 C CNN
@@
 ToF
 $Comp
-L PWR_FLAG #FLG063
+L PWR_FLAG #FLG068
 U 1 1 592CE2A7
 P 5300 2300
-F 0 "#FLG063" H 5300 2395 50  0001 C CNN
+F 0 "#FLG068" H 5300 2395 50  0001 C CNN
 F 1 "PWR_FLAG" H 5300 2480 50  0000 C CNN
 F 2 "" H 5300 2300 50  0000 C CNN
@@
 $EndComp
 $Comp
-L PWR_FLAG #FLG064
+L PWR_FLAG #FLG069
 U 1 1 592CE368
 P 5300 2600
-F 0 "#FLG064" H 5300 2695 50  0001 C CNN
+F 0 "#FLG069" H 5300 2695 50  0001 C CNN
 F 1 "PWR_FLAG" H 5300 2780 50  0000 C CNN
 F 2 "" H 5300 2600 50  0000 C CNN

Commit message: 自動配線1残し
Parts:
- renumbered C29 to C28, C30 to C29, P20 to P12, P21 to P13, R22 to R23, R23 to R24
Changed lines of the file:
@@
 	5400 3400 5300 3400
 $Comp
-L C_Small C30
+L C_Small C29
 U 1 1 592BA26F
 P 3900 3800
-F 0 "C30" H 3910 3870 50  0000 L CNN
+F 0 "C29" H 3910 3870 50  0000 L CNN
 F 1 "0.1u" H 3910 3720 50  0000 L CNN
 F 2 "Capacitors_SMD:C_0201" H 3900 3800 50  0001 C CNN
@@
 $EndComp
 $Comp
-L C_Small C29
+L C_Small C28
 U 1 1 592BA2BF
 P 3600 3800
-F 0 "C29" H 3610 3870 50  0000 L CNN
+F 0 "C28" H 3610 3870 50  0000 L CNN
 F 1 "4.7u" H 3610 3720 50  0000 L CNN
 F 2 "Capacitors_SMD:C_0402" H 3600 3800 50  0001 C CNN
@@
 	5400 3300 5400 3400
 $Comp
-L CONN_01X04 P20
+L CONN_01X04 P12
 U 1 1 592AB778
 P 4600 2450
-F 0 "P20" H 4600 2700 50  0000 C CNN
+F 0 "P12" H 4600 2700 50  0000 C CNN
 F 1 "ToF_Host" V 4700 2450 50  0000 C CNN
 F 2 "mouse:STAND_PR_HOST" H 4600 2450 50  0001 C CNN
@@
 $EndComp
 $Comp
-L CONN_01X04 P21
+L CONN_01X04 P13
 U 1 1 592AB803
 P 5000 2450
-F 0 "P21" H 5000 2700 50  0000 C CNN
+F 0 "P13" H 5000 2700 50  0000 C CNN
 F 1 "ToF_Slave" V 5100 2450 50  0000 C CNN
 F 2 "mouse:STAND_PR_SLAVE" H 5000 2450 50  0001 C CNN
@@
 $EndComp
 $Comp
-L GND #PWR066
+L GND #PWR067
 U 1 1 592ABB63
 P 4300 2700
-F 0 "#PWR066" H 4300 2450 50  0001 C CNN
+F 0 "#PWR067" H 4300 2450 50  0001 C CNN
 F 1 "GND" H 4300 2550 50  0000 C CNN
 F 2 "" H 4300 2700 50  0000 C CNN
@@
 	4300 2600 4400 2600
 $Comp
-L +3.3V #PWR067
+L +3.3V #PWR068
 U 1 1 592ABB9F
 P 4300 2200
-F 0 "#PWR067" H 4300 2050 50  0001 C CNN
+F 0 "#PWR068" H 4300 2050 50  0001 C CNN
 F 1 "+3.3V" H 4300 2340 50  0000 C CNN
 F 2 "" H 4300 2200 50  0000 C CNN
@@
 ToF
 $Comp
-L PWR_FLAG #FLG068
+L PWR_FLAG #FLG069
 U 1 1 592CE2A7
 P 5300 2300
-F 0 "#FLG068" H 5300 2395 50  0001 C CNN
+F 0 "#FLG069" H 5300 2395 50  0001 C CNN
 F 1 "PWR_FLAG" H 5300 2480 50  0000 C CNN
 F 2 "" H 5300 2300 50  0000 C CNN
@@
 $EndComp
 $Comp
-L PWR_FLAG #FLG069
+L PWR_FLAG #FLG070
 U 1 1 592CE368
 P 5300 2600
-F 0 "#FLG069" H 5300 2695 50  0001 C CNN
+F 0 "#FLG070" H 5300 2695 50  0001 C CNN
 F 1 "PWR_FLAG" H 5300 2780 50  0000 C CNN
 F 2 "" H 5300 2600 50  0000 C CNN
@@
 $EndComp
 $Comp
-L R_Small R22
+L R_Small R23
 U 1 1 5932174C
 P 5800 3500
-F 0 "R22" H 5830 3520 50  0000 L CNN
+F 0 "R23" H 5830 3520 50  0000 L CNN
 F 1 "4.7k" H 5830 3460 50  0000 L CNN
 F 2 "Resistors_SMD:R_0201" H 5800 3500 50  0001 C CNN
@@
 $EndComp
 $Comp
-L R_Small R23
+L R_Small R24
 U 1 1 593217CA
 P 6100 3500
-F 0 "R23" H 6130 3520 50  0000 L CNN
+F 0 "R24" H 6130 3520 50  0000 L CNN
 F 1 "4.7k" H 6130 3460 50  0000 L CNN
 F 2 "Resistors_SMD:R_0201" H 6100 3500 50  0001 C CNN

Commit message: 実装経験をもとにフットプリントを改良，ミスを修正
SC70サイズのオペアンプのピンアサインを修正
Parts:
- renumbered P12 to P11, P13 to P12
Changed lines of the file:
@@
 	5400 3300 5400 3400
 $Comp
-L CONN_01X04 P12
+L CONN_01X04 P11
 U 1 1 592AB778
 P 4600 2450
-F 0 "P12" H 4600 2700 50  0000 C CNN
+F 0 "P11" H 4600 2700 50  0000 C CNN
 F 1 "ToF_Host" V 4700 2450 50  0000 C CNN
 F 2 "mouse:STAND_PR_HOST" H 4600 2450 50  0001 C CNN
@@
 $EndComp
 $Comp
-L CONN_01X04 P13
+L CONN_01X04 P12
 U 1 1 592AB803
 P 5000 2450
-F 0 "P13" H 5000 2700 50  0000 C CNN
+F 0 "P12" H 5000 2700 50  0000 C CNN
 F 1 "ToF_Slave" V 5100 2450 50  0000 C CNN
 F 2 "mouse:STAND_PR_SLAVE" H 5000 2450 50  0001 C CNN
@@
 $EndComp
 $Comp
-L GND #PWR067
+L GND #PWR60
 U 1 1 592ABB63
 P 4300 2700
-F 0 "#PWR067" H 4300 2450 50  0001 C CNN
+F 0 "#PWR60" H 4300 2450 50  0001 C CNN
 F 1 "GND" H 4300 2550 50  0000 C CNN
 F 2 "" H 4300 2700 50  0000 C CNN
@@
 	4300 2600 4400 2600
 $Comp
-L +3.3V #PWR068
+L +3.3V #PWR59
 U 1 1 592ABB9F
 P 4300 2200
-F 0 "#PWR068" H 4300 2050 50  0001 C CNN
+F 0 "#PWR59" H 4300 2050 50  0001 C CNN
 F 1 "+3.3V" H 4300 2340 50  0000 C CNN
 F 2 "" H 4300 2200 50  0000 C CNN
@@
 ToF
 $Comp
-L PWR_FLAG #FLG069
+L PWR_FLAG #FLG9
 U 1 1 592CE2A7
 P 5300 2300
-F 0 "#FLG069" H 5300 2395 50  0001 C CNN
+F 0 "#FLG9" H 5300 2395 50  0001 C CNN
 F 1 "PWR_FLAG" H 5300 2480 50  0000 C CNN
 F 2 "" H 5300 2300 50  0000 C CNN
@@
 $EndComp
 $Comp
-L PWR_FLAG #FLG070
+L PWR_FLAG #FLG10
 U 1 1 592CE368
 P 5300 2600
-F 0 "#FLG070" H 5300 2695 50  0001 C CNN
+F 0 "#FLG10" H 5300 2695 50  0001 C CNN
 F 1 "PWR_FLAG" H 5300 2780 50  0000 C CNN
 F 2 "" H 5300 2600 50  0000 C CNN
